File: summer_2022_refurb/VCF_VCA_board/output_buffer.kicad_sch (KiCad schematic)
At the start: 5 parts

Commit message: Progress on refurb boards, all incomplete and messy still
Parts:
- removed C?: 10p, symbol Device:C
- removed R? (x2): 100k, symbol Device:R
- removed R?: 82k, symbol Device:R
- removed U?: TL072, symbol Amplifier_Operational:TL072
- added C?: 10p, symbol Device:C
- added R? (x3): 100k, symbol Device:R
- added U?: TL072, symbol Amplifier_Operational:TL072
Connections:
- net GND: now also U?.3 (+)
- net OUT: now also C?.2, R?.2, U?.1
- new net: C?.1, R?.1, R?.2, R?.2, U?.2 (-)
- new net IN_1: R?.1
- new net IN_2: R?.1
Other:
- title: Josh Ox Ribbon Synth VCF/VCA board -> (none)
