File: summer_2022_refurb/main_VCO_board/PWM_mixer.kicad_sch (KiCad schematic)
At the start: 0 parts

Commit message: Progress on refurb boards, all incomplete and messy still
Parts:
- added C?: 100p, symbol Device:C
- added R? (x6): 100k, symbol Device:R
- added RV? (x5): 100k, symbol Device:R_Potentiometer
- added U?: TL072, symbol Amplifier_Operational:TL072
Connections:
- new net: C?.1, R?.1, R?.2, R?.2, R?.2, R?.2, R?.2, U?.2 (-)
- new net: C?.2, R?.2, U?.1
- new net: R?.1, RV?.2 (x5)
- new net GND: RV?.1, RV?.1, RV?.1, RV?.1, RV?.1, U?.3 (+)
