File: summer_2022_refurb/main_VCO_board/harmonic_pulse_shaper.kicad_sch (KiCad schematic)
At the start: 32 parts

Commit message: Progress on refurb boards, all incomplete and messy still
Parts:
- removed R?: 100k, symbol Device:R
- R?: value 100k -> 120k
- R?: value R -> ?
Connections:
- net -5VA renamed -5V_REF
- net CV_IN_2 renamed PWM_IN
Other:
- note added: "needs lots of work, check everything"
- moved on the sheet: R?
Changed lines of the file:
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@@
   (junction (at 204.47 109.22) (diameter 0) (color 0 0 0 0)
   )
-  (junction (at 92.71 165.1) (diameter 0) (color 0 0 0 0)
-  )
   (junction (at 181.61 110.49) (diameter 0) (color 0 0 0 0)
   )
@@
     (stroke (width 0) (type default) (color 0 0 0 0))
   )
-  (wire (pts (xy 92.71 154.94) (xy 92.71 165.1))
-    (stroke (width 0) (type default) (color 0 0 0 0))
-  )
   (wire (pts (xy 240.03 99.06) (xy 233.68 99.06))
     (stroke (width 0) (type default) (color 0 0 0 0))
@@
     (stroke (width 0) (type default) (color 0 0 0 0))
   )
-  (wire (pts (xy 80.01 165.1) (xy 82.55 165.1))
+  (wire (pts (xy 80.01 160.02) (xy 82.55 160.02))
     (stroke (width 0) (type default) (color 0 0 0 0))
   )
@@
     (stroke (width 0) (type default) (color 0 0 0 0))
   )
-  (wire (pts (xy 92.71 170.18) (xy 92.71 165.1))
-    (stroke (width 0) (type default) (color 0 0 0 0))
-  )
-  (wire (pts (xy 90.17 154.94) (xy 92.71 154.94))
+  (wire (pts (xy 92.71 170.18) (xy 92.71 160.02))
     (stroke (width 0) (type default) (color 0 0 0 0))
   )
@@
     (stroke (width 0) (type default) (color 0 0 0 0))
   )
-  (wire (pts (xy 90.17 165.1) (xy 92.71 165.1))
+  (wire (pts (xy 90.17 160.02) (xy 92.71 160.02))
     (stroke (width 0) (type default) (color 0 0 0 0))
   )
@@
     (stroke (width 0) (type default) (color 0 0 0 0))
   )
-  (wire (pts (xy 80.01 154.94) (xy 82.55 154.94))
-    (stroke (width 0) (type default) (color 0 0 0 0))
-  )
   (wire (pts (xy 127 170.18) (xy 129.54 170.18))
     (stroke (width 0) (type default) (color 0 0 0 0))
@@
     (stroke (width 0) (type default) (color 0 0 0 0))
   )
-  (wire (pts (xy 80.01 176.53) (xy 80.01 173.99))
-    (stroke (width 0) (type default) (color 0 0 0 0))
-  )
   (wire (pts (xy 233.68 87.63) (xy 240.03 87.63))
     (stroke (width 0) (type default) (color 0 0 0 0))
@@
     (stroke (width 0) (type default) (color 0 0 0 0))
   )
-  (hierarchical_label "CV_IN_1" (shape input) (at 80.01 154.94 180)
+  (text "needs lots of work,\ncheck everything" (at 127 50.8 0)
+    (effects (font (size 3 3)) (justify left bottom))
+  )
+  (global_label "-5V_REF" (shape input) (at 80.01 173.99 180) (fields_autoplaced)
     (effects (font (size 1.27 1.27)) (justify right))
+    (property "Intersheet References" "${INTERSHEET_REFS}" (id 0) (at 69.2512 173.9106 0)
+      (effects (font (size 1.27 1.27)) (justify right) hide)
+    )
   )
   (hierarchical_label "SIGNAL_IN" (shape input) (at 52.07 88.9 180)
@@
     (effects (font (size 1.27 1.27)) (justify left))
   )
-  (hierarchical_label "CV_IN_2" (shape input) (at 80.01 165.1 180)
+  (hierarchical_label "PWM_IN" (shape input) (at 80.01 160.02 180)
     (effects (font (size 1.27 1.27)) (justify right))
   )
@@
     )
     (property "Datasheet" "~" (id 3) (at 194.31 88.9 0)
-      (effects (font (size 1.27 1.27)) hide)
-    )
-    (pin "1")
-    (pin "2")
-  )
-  (symbol (lib_id "Device:R") (at 86.36 154.94 90) (unit 1)
-    (in_bom yes) (on_board yes) (fields_autoplaced)
-    (property "Reference" "R?" (id 0) (at 86.36 148.59 90))
-    (property "Value" "100k" (id 1) (at 86.36 151.13 90))
-    (property "Footprint" "" (id 2) (at 86.36 156.718 90)
-      (effects (font (size 1.27 1.27)) hide)
-    )
-    (property "Datasheet" "~" (id 3) (at 86.36 154.94 0)
       (effects (font (size 1.27 1.27)) hide)
     )
@@
     (pin "2")
   )
-  (symbol (lib_id "Device:R") (at 86.36 165.1 90) (unit 1)
-    (in_bom yes) (on_board yes) (fields_autoplaced)
-    (property "Reference" "R?" (id 0) (at 86.36 158.75 90))
-    (property "Value" "100k" (id 1) (at 86.36 161.29 90))
-    (property "Footprint" "" (id 2) (at 86.36 166.878 90)
-      (effects (font (size 1.27 1.27)) hide)
-    )
-    (property "Datasheet" "~" (id 3) (at 86.36 165.1 0)
+  (symbol (lib_id "Device:R") (at 86.36 160.02 90) (unit 1)
+    (in_bom yes) (on_board yes) (fields_autoplaced)
+    (property "Reference" "R?" (id 0) (at 86.36 153.67 90))
+    (property "Value" "120k" (id 1) (at 86.36 156.21 90))
+    (property "Footprint" "" (id 2) (at 86.36 161.798 90)
+      (effects (font (size 1.27 1.27)) hide)
+    )
+    (property "Datasheet" "~" (id 3) (at 86.36 160.02 0)
       (effects (font (size 1.27 1.27)) hide)
     )
@@
     (in_bom yes) (on_board yes) (fields_autoplaced)
     (property "Reference" "R?" (id 0) (at 86.36 167.64 90))
-    (property "Value" "R" (id 1) (at 86.36 170.18 90))
+    (property "Value" "?" (id 1) (at 86.36 170.18 90))
     (property "Footprint" "" (id 2) (at 86.36 175.768 90)
       (effects (font (size 1.27 1.27)) hide)
@@
     (pin "8")
   )
-  (symbol (lib_id "power:-5VA") (at 80.01 176.53 180) (unit 1)
-    (in_bom yes) (on_board yes) (fields_autoplaced)
-    (property "Reference" "#PWR?" (id 0) (at 80.01 179.07 0)
-      (effects (font (size 1.27 1.27)) hide)
-    )
-    (property "Value" "-5VA" (id 1) (at 80.01 181.61 0))
-    (property "Footprint" "" (id 2) (at 80.01 176.53 0)
-      (effects (font (size 1.27 1.27)) hide)
-    )
-    (property "Datasheet" "" (id 3) (at 80.01 176.53 0)
-      (effects (font (size 1.27 1.27)) hide)
-    )
-    (pin "1")
-  )
   (symbol (lib_id "Device:R") (at 105.41 160.02 90) (unit 1)
