File: summer_2022_refurb/main_VCO_board/lin_FM_conditioner.kicad_sch (KiCad schematic)
At the start: 17 parts

Commit message: Progress on refurb boards, all incomplete and messy still
Connections:
- net +2V5 renamed +2V5_REF
Changed lines of the file:
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@@
-    (stroke (width 0) (type default) (color 0 0 0 0))
-  )
-  (wire (pts (xy 77.47 68.58) (xy 77.47 72.39))
     (stroke (width 0) (type default) (color 0 0 0 0))
   )
@@
   (wire (pts (xy 93.98 86.36) (xy 91.44 86.36))
     (stroke (width 0) (type default) (color 0 0 0 0))
+  )
+  (global_label "+2V5_REF" (shape input) (at 77.47 72.39 180) (fields_autoplaced)
+    (effects (font (size 1.27 1.27)) (justify right))
+    (property "Intersheet References" "${INTERSHEET_REFS}" (id 0) (at 65.5017 72.3106 0)
+      (effects (font (size 1.27 1.27)) (justify right) hide)
+    )
   )
   (hierarchical_label "LIN_FM_IN" (shape input) (at 67.31 86.36 180)
@@
     (pin "2")
   )
-  (symbol (lib_id "power:+2V5") (at 77.47 68.58 0) (unit 1)
-    (in_bom yes) (on_board yes) (fields_autoplaced)
-    (property "Reference" "#PWR?" (id 0) (at 77.47 72.39 0)
-      (effects (font (size 1.27 1.27)) hide)
-    )
-    (property "Value" "+2V5" (id 1) (at 77.47 63.5 0))
-    (property "Footprint" "" (id 2) (at 77.47 68.58 0)
-      (effects (font (size 1.27 1.27)) hide)
-    )
-    (property "Datasheet" "" (id 3) (at 77.47 68.58 0)
-      (effects (font (size 1.27 1.27)) hide)
-    )
-    (pin "1")
-  )
   (symbol (lib_id "power:GND") (at 187.96 110.49 0) (unit 1)
