File: summer_2022_refurb/main_VCO_board/saw_animator.kicad_sch (KiCad schematic)
At the start: 26 parts

Commit message: Progress on refurb boards, all incomplete and messy still
Parts:
- removed R? (x2): 200k, symbol Device:R
- removed R? (x2): R, symbol Device:R
- removed R? (x2): 100k, symbol Device:R
- removed U?: TL072, symbol Amplifier_Operational:TL072
- added C?: 100p, symbol Device:C
- added C?: 10u, symbol Device:C
- added R?: 1k, symbol Device:R
- added R?: 2k7, symbol Device:R
- added R?: 8k2, symbol Device:R
- added R?: 51k, symbol Device:R
- C?: value C -> ?
- R?: value 100k -> ?
- R?: value R -> ?
- R?: value 47k -> 180k
- R?: value 330k -> 1M
- R?: value 100k -> 200k
- RV?: value 10k -> 50k
Connections:
- net +12V is gone; now on net +5V: U?.8 (V+)
- net -12V is gone; now on net GND: U?.4 (V-)
- net +5V: now also R?.1
- net GND: now also C?.2, R?.2; no longer U?.2 (-), U?.3 (+)
- net SAW_IN: now also R?.1, R?.1
- net RATE_R_2: now reaches C?.1, U?.2 (-)
- net RATE_R_1: now reaches R?.2
- net at R?.1, RV?.1, U?.7: now also R?.2
- net +/-5v saw: no longer names the net of U?.2 (+)
- net +/-5v saw: now also C?.1, R?.2; no longer R?.1
- new net: C?.1, R?.1, R?.2, U?.2 (-), U?.3 (+)
- new net: C?.2, R?.1
Other:
- note added: "DC offset trim Adjust for minimal glitch in the triangle wave which is fed from the sawtooth output."
- note added: "NOT DONE"
- note added: "Resistor at this node sets the LFO frequency"
- note added: "Triangle LFO [0, +2.5v]"
- note added: "Upgoing sawtooth [-1.25, +1.25v]"
- note added: "Upgoing sawtooth [0, +2.5v]"
- note removed: "DC offset trim Adjust for minimal DC offset at the saw output. Note that this trimmer will have a large impact on the triangle wave."
- moved on the sheet: C?, R?, U?A
