File: summer_2022_refurb/sample_and_hold_board/sample_and_hold_board.kicad_sch (KiCad schematic)
At the start: 0 parts

Commit message: Initial S&H board layout
Parts:
- added J1: VCO_port, Connector_Molex:Molex_KK-254_AE-6410-06A_1x06_P2.54mm_Vertical, symbol Connector_Generic:Conn_01x06
- added J2: VCF_port, Connector_Molex:Molex_KK-254_AE-6410-03A_1x03_P2.54mm_Vertical, symbol Connector_Generic:Conn_01x03
- added J3: ribbon_port, Connector_Molex:Molex_KK-254_AE-6410-02A_1x02_P2.54mm_Vertical, symbol Connector_Generic:Conn_01x02
- added TP1: S&H mixer, TestPoint:TestPoint_Keystone_5000-5004_Miniature, symbol Connector:TestPoint
- added TP2: S&H, TestPoint:TestPoint_Keystone_5000-5004_Miniature, symbol Connector:TestPoint
- added TP3: trigger, TestPoint:TestPoint_Keystone_5000-5004_Miniature, symbol Connector:TestPoint
Connections:
- net noise_generator/NOISE_OUT: now also J1.3 (Pin_3)
- net s&h_mixer/MAIN_VCO: now also J1.4 (Pin_4)
- net s&h_mixer/PWM_LFO: now also J1.5 (Pin_5)
- net sample_and_hold/TRIGGER_IN: now also J3.2 (Pin_2), TP3.1
- new net GND: J1.6 (Pin_6), J2.3 (Pin_3), J3.1 (Pin_1)
- new net S&H: J1.1 (Pin_1), J2.1 (Pin_1), TP2.1
- new net S&H_MIXER: J1.2 (Pin_2), J2.2 (Pin_2), TP1.1
Other:
- added sheet power_supply (power_supply.kicad_sch)
- title: (none) -> Josh Ox Ribbon Synth Sample and Hold Board
