File: summer_2022_refurb/mod_osc_board/VCO_core.kicad_sch (KiCad schematic)
At the start: 43 parts

Commit message: Modosc schem progress
Parts:
- removed R?: 100K, symbol Device:R
- gave numbers to parts that had none: 37
Other:
- title: (none) -> Josh Ox Ribbon Synth Mod Osc board

Commit message: Initial mod osc layout
Parts:
- removed SW201: SW_Rotary5, symbol custom_symbols:SW_Rotary5
- added SW201: alpha_SR2612F-0112, custom_footprints:apha_SR2612F-0112, symbol custom_symbols:alpha_SR2612F-0112
- C201, C202, C203, C204: footprint (none) -> Capacitor_SMD:C_0805_2012Metric
- R201, R202, R203, R204, R205, R206, R207, R208, R209, R210, R211, R212, R213, R214, R215, R216, R217, R218, R219, R220, R221, R222, R223, R224, R225: footprint (none) -> Resistor_SMD:R_0805_2012Metric
- RV201, RV202, RV203: footprint (none) -> Potentiometer_THT:Potentiometer_Bourns_3296W_Vertical
- U201: footprint (none) -> custom_footprints:PQN32_HandSoldering
- U202: footprint (none) -> Package_SO:SO-8_5.3x6.2mm_P1.27mm
Connections:
- net at U201.12 (aux_1_mix): now also SW201.1
- net at U201.9 (tri_mix): now also SW201.2
- net at U201.10 (saw_mix): now also SW201.3
- net at U201.13 (aux_2_mix): now also SW201.4
- net at U201.11 (pulse_mix): now also SW201.5
- net at R219.2: now also SW201.13
- net -5V_REF renamed -5V
- no-connect marks 3 -> 10
Other:
- moved on the sheet: C203, R202, R203, R204, R205, R206, R207, R211, R212, R219, R221, R225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
