File: summer_2022_refurb/ADSR_board/ADSR_board.kicad_pcb (KiCad board)
At the start: 2 copper layers, 175.3 x 111.8 mm, 214 parts, among them J1 ribbon_port, J2 modosc_port, J3 VCO_port, J4 VCF_port, J5 power_entry, Q201 MMBT3904, Q202 MMBT3904, Q203 MMBT3906, Q204 MMBT3904, Q205 MMBT3906, Q206 MMBT3904, Q207 MMBT3904, Q208 MMBT3906, Q209 MMBT3904, Q210 MMBT3904, Q211 MMBT3904, Q212 MMBT3904, Q301 MMBT3904, Q302 MMBT3904, Q303 MMBT3906, Q304 MMBT3904, Q305 MMBT3906, Q306 MMBT3904, Q307 MMBT3904, Q308 MMBT3906, Q309 MMBT3904, Q310 MMBT3904, Q311 MMBT3904, Q312 MMBT3904, Q401 MMBT3904, Q402 MMBT3904, Q403 MMBT3906, Q404 MMBT3904, Q405 MMBT3906, Q406 MMBT3904, Q407 MMBT3904, Q408 MMBT3906, Q409 MMBT3904, Q410 MMBT3904, Q411 MMBT3904, Q412 MMBT3904, SW201 SW_SPDT, SW301 SW_SPDT, SW401 SW_SPDT, U201 TL072, U202 TL072, U301 TL072, U302 TL072, U401 TL072, U402 TL072

Commit message: Initial ADSR board layout, 555 version
Parts:
- removed C514, C515, C516, C517, C518, C519, C520: 100n, Capacitor_SMD:C_0805_2012Metric
- removed Q205, Q208, Q305, Q308, Q405, Q408: MMBT3906, Package_TO_SOT_SMD:SOT-23
- removed Q206, Q207, Q209, Q210, Q211, Q212, Q306, Q307, Q309, Q310, Q311, Q312, Q406, Q407, Q409, Q410, Q411, Q412: MMBT3904, Package_TO_SOT_SMD:SOT-23
- removed R212, R312, R412: 1k, Resistor_SMD:R_0805_2012Metric
- removed R213, R313, R413: 3k9, Resistor_SMD:R_0805_2012Metric
- removed R214, R314, R414: 4k7, Resistor_SMD:R_0805_2012Metric
- removed R215, R218, R220, R229, R232, R235, R315, R318, R320, R329, R332, R335, R415, R418, R420, R429, R432, R435: 10k, Resistor_SMD:R_0805_2012Metric
- removed R216, R316, R416: 470, Resistor_SMD:R_0805_2012Metric
- removed R217, R317, R417: 82k, Resistor_SMD:R_0805_2012Metric
- removed R219, R221, R225, R233, R319, R321, R325, R333, R419, R421, R425, R433: 33k, Resistor_SMD:R_0805_2012Metric
- removed R222, R322, R422: 47k, Resistor_SMD:R_0805_2012Metric
- removed R223, R224, R226, R228, R234, R323, R324, R326, R328, R334, R423, R424, R426, R428, R434: 100k, Resistor_SMD:R_0805_2012Metric
- removed R227, R327, R427: 8k2, Resistor_SMD:R_0805_2012Metric
- removed R230, R330, R430: 15k, Resistor_SMD:R_0805_2012Metric
- removed R231, R331, R431: 1M, Resistor_SMD:R_0805_2012Metric
- added D205: 1N4148W, Diode_SMD:D_SOD-123, B.Cu at (44.5, 35.6)
- added D305: 1N4148W, Diode_SMD:D_SOD-123, B.Cu at (277.8, 87.6)
- added D405: 1N4148W, Diode_SMD:D_SOD-123, B.Cu at (275.3, 151.1)
- added R101: 1k, Resistor_SMD:R_0805_2012Metric, B.Cu at (21.6, 171.8)
- added R102: 1k, Resistor_SMD:R_0805_2012Metric, B.Cu at (30.3, 179.6)
- added R103: 100k, Resistor_SMD:R_0805_2012Metric, B.Cu at (34.7, 179.6)
- added R104: 1k, Resistor_SMD:R_0805_2012Metric, B.Cu at (26.0, 171.8)
- added R105: 100k, Resistor_SMD:R_0805_2012Metric, B.Cu at (39.1, 179.5)
- added R106: 1k, Resistor_SMD:R_0805_2012Metric, B.Cu at (26.0, 174.7)
- added R107: 1k, Resistor_SMD:R_0805_2012Metric, B.Cu at (43.6, 179.5)
- added U101: TL072, Package_SO:SO-8_5.3x6.2mm_P1.27mm, B.Cu at (40.5, 174.2)
- C201, C301, C401: value 100n -> 10n; footprint Capacitor_THT:C_Rect_L7.2mm_W3.0mm_P5.00mm_FKS2_FKP2_MKS2_MKP2 -> Capacitor_SMD:C_0805_2012Metric
- C202, C302, C402: value 47n -> 2u2; footprint Capacitor_THT:C_Rect_L7.2mm_W3.0mm_P5.00mm_FKS2_FKP2_MKS2_MKP2 -> Capacitor_THT:CP_Radial_D6.3mm_P2.50mm
- C203, C303, C403: value 10p -> 22u; footprint Capacitor_SMD:C_0805_2012Metric -> Capacitor_THT:CP_Radial_D6.3mm_P2.50mm
- C204, C304, C404: value 1n -> 10n
- C502: value 100n -> 10u; footprint Capacitor_SMD:C_0805_2012Metric -> Capacitor_THT:CP_Radial_D6.3mm_P2.50mm
- C511: value 10u -> 100n; footprint Capacitor_THT:CP_Radial_D6.3mm_P2.50mm -> Capacitor_SMD:C_0805_2012Metric
- Q201, Q301, Q401: value MMBT3904 -> 2N7002
- Q203, Q303, Q403: value MMBT3906 -> MMBT3904
- R201, R301, R401: value 110k -> 4k7
- R202, R302, R402: value 680k -> 1M
- R203, R303, R403: value 2k7 -> R
- R204, R304, R404: value 110k -> 10k
- R205, R305, R405: value 18k -> 10k
- R206, R306, R406: value 1M -> 10k
- R207, R307, R407: value 390k -> R
- R208, R308, R408: value 2k7 -> 10k
- R210, R310, R410: value 1M -> R
- R211, R311, R411: value 68k -> 22
- RV201, RV202, RV204, RV301, RV302, RV304, RV401, RV402, RV404: value 100k -> 500kA
- RV203, RV303, RV403: value 100k -> 10k
- U202, U302, U402: value TL072 -> LM555xM; footprint Package_SO:SO-8_5.3x6.2mm_P1.27mm -> Package_SO:SOIC-8_3.9x4.9mm_P1.27mm
- moved D303 219.8 mm to (272.1, 91.0)
- moved D302 207.7 mm to (277.8, 91.0)
- moved R301 205.6 mm to (234.3, 63.0)
- moved D301 205.3 mm to (272.1, 87.6)
- moved R308 195.4 mm to (252.4, 81.4)
- moved R303 194.0 mm to (241.2, 70.4)
- moved D304 193.4 mm to (238.1, 59.9)
- moved C304 193.0 mm to (238.7, 63.1)
- moved R307 192.2 mm to (241.2, 67.4)
- moved U302 188.0 mm to (284.9, 89.2)
- moved R302 186.7 mm to (228.6, 59.7)
- moved Q301 177.8 mm to (261.9, 88.2)
- moved R304 165.1 mm to (236.8, 66.0)
- moved R306 163.7 mm to (252.4, 84.3)
- moved R305 140.4 mm to (257.2, 85.8)
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Connections:
- C202 pad 1: Net-(C201-Pad1) -> Net-(C202-Pad1)
- C202 pad 2: /modulation_ADSR/OUT -> GND
- C203 pad 1: Net-(C203-Pad1) -> Net-(C202-Pad1)
- C204 pad 2: Net-(C204-Pad2) -> GND
- C302 pad 1: Net-(C301-Pad1) -> Net-(C302-Pad1)
- C302 pad 2: /VCF_ADSR/OUT -> GND
- C303 pad 1: Net-(C303-Pad1) -> Net-(C302-Pad1)
- C304 pad 2: Net-(C304-Pad2) -> GND
- C402 pad 1: Net-(C401-Pad1) -> Net-(C402-Pad1)
- C402 pad 2: /VCA_ENV -> GND
- C403 pad 1: Net-(C403-Pad1) -> Net-(C402-Pad1)
- C404 pad 2: Net-(C404-Pad2) -> GND
- C502 pad 1: +15V -> GND
- C502 pad 2: GND -> -15V
- C504 pad 1: +15V -> GND
- C504 pad 2: GND -> -15V
- C506 pad 1: +15V -> GND
- C506 pad 2: GND -> -15V
- C508 pad 1: +15V -> GND
- C508 pad 2: GND -> -15V
- C510 pad 1: +15V -> GND
- C510 pad 2: GND -> -15V
- C511 pad 1: GND -> +15V
- C511 pad 2: -15V -> GND
- C512 pad 1: GND -> +15V
- C512 pad 2: -15V -> GND
- C513 pad 1: GND -> +15V
- C513 pad 2: -15V -> GND
- D201 pad 2: Net-(D201-Pad2) -> Net-(C202-Pad1)
- D202 pad 1: Net-(D202-Pad1) -> Net-(C202-Pad1)
- D202 pad 2: Net-(D201-Pad1) -> Net-(D202-Pad2)
- D203 pad 2: Net-(D202-Pad1) -> Net-(C202-Pad1)
- D204 pad 1: Net-(D203-Pad1) -> Net-(C201-Pad2)
- D204 pad 2: Net-(D204-Pad2) -> GND
- D301 pad 2: Net-(D301-Pad2) -> Net-(C302-Pad1)
- D302 pad 1: Net-(D302-Pad1) -> Net-(C302-Pad1)
- D302 pad 2: Net-(D301-Pad1) -> Net-(D302-Pad2)
- D303 pad 2: Net-(D302-Pad1) -> Net-(C302-Pad1)
- D304 pad 1: Net-(D303-Pad1) -> Net-(C301-Pad2)
- D304 pad 2: Net-(D304-Pad2) -> GND
- D401 pad 2: Net-(D401-Pad2) -> Net-(C402-Pad1)
- D402 pad 1: Net-(D402-Pad1) -> Net-(C402-Pad1)
- D402 pad 2: Net-(D401-Pad1) -> Net-(D402-Pad2)
- D403 pad 2: Net-(D402-Pad1) -> Net-(C402-Pad1)
- D404 pad 1: Net-(D403-Pad1) -> Net-(C401-Pad2)
- D404 pad 2: Net-(D404-Pad2) -> GND
- J1 pad 1: /MOD_ENV_GATE -> /modulation_ADSR/GATE
- J1 pad 2: /VCF_ENV_GATE -> /VCF_ADSR/GATE
- J1 pad 3: /VCA_ENV_GATE -> /VCA_ADSR/GATE
- J2 pad 1: /modulation_ADSR/OUT -> Net-(J2-Pad1)
- J3 pad 1: /modulation_ADSR/OUT -> Net-(J3-Pad1)
- J3 pad 2: /modulation_ADSR/INVERTING_OUT -> Net-(J3-Pad2)
- J4 pad 1: /VCF_ADSR/OUT -> Net-(J4-Pad1)
- Q202 pad 3: Net-(C203-Pad1) -> Net-(C201-Pad1)
- Q203 pad 1: Net-(Q201-Pad2) -> Net-(Q203-Pad1)
- Q203 pad 2: Net-(Q202-Pad2) -> GND
- Q203 pad 3: Net-(C201-Pad1) -> Net-(Q203-Pad3)
- Q204 pad 1: Net-(Q204-Pad1) -> Net-(D205-Pad1)
- Q204 pad 2: Net-(Q201-Pad2) -> Net-(Q202-Pad2)
- Q204 pad 3: Net-(Q204-Pad3) -> Net-(Q202-Pad1)
- Q302 pad 3: Net-(C303-Pad1) -> Net-(C301-Pad1)
- Q303 pad 1: Net-(Q301-Pad2) -> Net-(Q303-Pad1)
- Q303 pad 2: Net-(Q302-Pad2) -> GND
- Q303 pad 3: Net-(C301-Pad1) -> Net-(Q303-Pad3)
- Q304 pad 1: Net-(Q304-Pad1) -> Net-(D305-Pad1)
- Q304 pad 2: Net-(Q301-Pad2) -> Net-(Q302-Pad2)
- Q304 pad 3: Net-(Q304-Pad3) -> Net-(Q302-Pad1)
- Q402 pad 3: Net-(C403-Pad1) -> Net-(C401-Pad1)
- Q403 pad 1: Net-(Q401-Pad2) -> Net-(Q403-Pad1)
- Q403 pad 2: Net-(Q402-Pad2) -> GND
- Q403 pad 3: Net-(C401-Pad1) -> Net-(Q403-Pad3)
- Q404 pad 1: Net-(Q404-Pad1) -> Net-(D405-Pad1)
- Q404 pad 2: Net-(Q401-Pad2) -> Net-(Q402-Pad2)
- Q404 pad 3: Net-(Q404-Pad3) -> Net-(Q402-Pad1)
- R201 pad 1: /modulation_ADSR/ATTACK_CV -> +15V
- R201 pad 2: Net-(Q202-Pad1) -> Net-(R201-Pad2)
- R202 pad 1: Net-(Q202-Pad1) -> Net-(C201-Pad1)
- R202 pad 2: -15V -> Net-(Q201-Pad1)
- R203 pad 1: Net-(Q202-Pad1) -> Net-(R203-Pad1)
- R203 pad 2: GND -> Net-(D201-Pad1)
- R204 pad 1: /modulation_ADSR/DECAY_CV -> +15V
- R204 pad 2: Net-(Q201-Pad3) -> Net-(Q202-Pad1)
- R205 pad 1: /modulation_ADSR/SUSTAIN_CV -> +15V
- R205 pad 2: Net-(Q207-Pad3) -> Net-(C201-Pad1)
- R206 pad 1: Net-(Q201-Pad1) -> +15V
- R206 pad 2: Net-(Q210-Pad3) -> Net-(Q203-Pad3)
- R207 pad 1: Net-(Q201-Pad2) -> Net-(R207-Pad1)
- R207 pad 2: -15V -> Net-(D202-Pad2)
- R208 pad 1: Net-(Q201-Pad2) -> Net-(C201-Pad2)
- R208 pad 2: GND -> Net-(Q203-Pad1)
- R209 pad 1: /modulation_ADSR/RELEASE_CV -> /modulation_ADSR/GATE
- R209 pad 2: Net-(Q204-Pad3) -> Net-(D205-Pad1)
- R210 pad 1: Net-(Q204-Pad1) -> Net-(D203-Pad1)
- R210 pad 2: Net-(D202-Pad1) -> Net-(R210-Pad2)
- R211 pad 1: Net-(D202-Pad1) -> Net-(Q202-Pad2)
- R211 pad 2: Net-(Q207-Pad1) -> GND
- R301 pad 1: /VCF_ADSR/ATTACK_CV -> +15V
- R301 pad 2: Net-(Q302-Pad1) -> Net-(R301-Pad2)
- R302 pad 1: Net-(Q302-Pad1) -> Net-(C301-Pad1)
- R302 pad 2: -15V -> Net-(Q301-Pad1)
- R303 pad 1: Net-(Q302-Pad1) -> Net-(R303-Pad1)
- R303 pad 2: GND -> Net-(D301-Pad1)
- R304 pad 1: /VCF_ADSR/DECAY_CV -> +15V
- R304 pad 2: Net-(Q301-Pad3) -> Net-(Q302-Pad1)
- R305 pad 1: /VCF_ADSR/SUSTAIN_CV -> +15V
- R305 pad 2: Net-(Q307-Pad3) -> Net-(C301-Pad1)
- R306 pad 1: Net-(Q301-Pad1) -> +15V
- R306 pad 2: Net-(Q310-Pad3) -> Net-(Q303-Pad3)
- R307 pad 1: Net-(Q301-Pad2) -> Net-(R307-Pad1)
- R307 pad 2: -15V -> Net-(D302-Pad2)
- R308 pad 1: Net-(Q301-Pad2) -> Net-(C301-Pad2)
- R308 pad 2: GND -> Net-(Q303-Pad1)
- R309 pad 1: /VCF_ADSR/RELEASE_CV -> /VCF_ADSR/GATE
- R309 pad 2: Net-(Q304-Pad3) -> Net-(D305-Pad1)
- R310 pad 1: Net-(Q304-Pad1) -> Net-(D303-Pad1)
- R310 pad 2: Net-(D302-Pad1) -> Net-(R310-Pad2)
- R311 pad 1: Net-(D302-Pad1) -> Net-(Q302-Pad2)
- R311 pad 2: Net-(Q307-Pad1) -> GND
- R401 pad 1: /VCA_ADSR/ATTACK_CV -> +15V
- R401 pad 2: Net-(Q402-Pad1) -> Net-(R401-Pad2)
- R402 pad 1: Net-(Q402-Pad1) -> Net-(C401-Pad1)
- R402 pad 2: -15V -> Net-(Q401-Pad1)
- R403 pad 1: Net-(Q402-Pad1) -> Net-(R403-Pad1)
- R403 pad 2: GND -> Net-(D401-Pad1)
- R404 pad 1: /VCA_ADSR/DECAY_CV -> +15V
- R404 pad 2: Net-(Q401-Pad3) -> Net-(Q402-Pad1)
- R405 pad 1: /VCA_ADSR/SUSTAIN_CV -> +15V
- R405 pad 2: Net-(Q407-Pad3) -> Net-(C401-Pad1)
- R406 pad 1: Net-(Q401-Pad1) -> +15V
- R406 pad 2: Net-(Q410-Pad3) -> Net-(Q403-Pad3)
- R407 pad 1: Net-(Q401-Pad2) -> Net-(R407-Pad1)
- R407 pad 2: -15V -> Net-(D402-Pad2)
- R408 pad 1: Net-(Q401-Pad2) -> Net-(C401-Pad2)
- R408 pad 2: GND -> Net-(Q403-Pad1)
- R409 pad 1: /VCA_ADSR/RELEASE_CV -> /VCA_ADSR/GATE
- R409 pad 2: Net-(Q404-Pad3) -> Net-(D405-Pad1)
- R410 pad 1: Net-(Q404-Pad1) -> Net-(D403-Pad1)
- R410 pad 2: Net-(D402-Pad1) -> Net-(R410-Pad2)
- R411 pad 1: Net-(D402-Pad1) -> Net-(Q402-Pad2)
- R411 pad 2: Net-(Q407-Pad1) -> GND
- RV201 pad 1: GND -> Net-(RV201-Pad1)
- RV201 pad 2: /modulation_ADSR/ATTACK_CV -> Net-(R207-Pad1)
- RV201 pad 3: +15V -> Net-(R207-Pad1)
- RV202 pad 1: GND -> Net-(R203-Pad1)
- RV202 pad 2: /modulation_ADSR/DECAY_CV -> Net-(RV202-Pad2)
- RV202 pad 3: +15V -> Net-(RV202-Pad2)
- RV203 pad 1: GND -> Net-(Q201-Pad3)
- RV203 pad 2: /modulation_ADSR/SUSTAIN_CV -> Net-(RV203-Pad2)
- RV203 pad 3: +15V -> Net-(R201-Pad2)
- RV204 pad 1: GND -> Net-(C201-Pad1)
- RV204 pad 2: /modulation_ADSR/RELEASE_CV -> Net-(R210-Pad2)
- RV204 pad 3: +15V -> Net-(R210-Pad2)
- RV301 pad 1: GND -> Net-(RV301-Pad1)
- RV301 pad 2: /VCF_ADSR/ATTACK_CV -> Net-(R307-Pad1)
- RV301 pad 3: +15V -> Net-(R307-Pad1)
- RV302 pad 1: GND -> Net-(R303-Pad1)
- RV302 pad 2: /VCF_ADSR/DECAY_CV -> Net-(RV302-Pad2)
- RV302 pad 3: +15V -> Net-(RV302-Pad2)
- RV303 pad 1: GND -> Net-(Q301-Pad3)
- RV303 pad 2: /VCF_ADSR/SUSTAIN_CV -> Net-(RV303-Pad2)
- RV303 pad 3: +15V -> Net-(R301-Pad2)
- RV304 pad 1: GND -> Net-(C301-Pad1)
- RV304 pad 2: /VCF_ADSR/RELEASE_CV -> Net-(R310-Pad2)
- RV304 pad 3: +15V -> Net-(R310-Pad2)
- RV401 pad 1: GND -> Net-(RV401-Pad1)
- RV401 pad 2: /VCA_ADSR/ATTACK_CV -> Net-(R407-Pad1)
- RV401 pad 3: +15V -> Net-(R407-Pad1)
- RV402 pad 1: GND -> Net-(R403-Pad1)
- RV402 pad 2: /VCA_ADSR/DECAY_CV -> Net-(RV402-Pad2)
- RV402 pad 3: +15V -> Net-(RV402-Pad2)
- RV403 pad 1: GND -> Net-(Q401-Pad3)
- RV403 pad 2: /VCA_ADSR/SUSTAIN_CV -> Net-(RV403-Pad2)
- RV403 pad 3: +15V -> Net-(R401-Pad2)
- RV404 pad 1: GND -> Net-(C401-Pad1)
- RV404 pad 2: /VCA_ADSR/RELEASE_CV -> Net-(R410-Pad2)
- RV404 pad 3: +15V -> Net-(R410-Pad2)
- SW201 pad 2: Net-(C201-Pad2) -> GND
- SW201 pad 3: /modulation_ADSR/OUT -> Net-(C203-Pad2)
- SW301 pad 2: Net-(C301-Pad2) -> GND
- SW301 pad 3: /VCF_ADSR/OUT -> Net-(C303-Pad2)
- SW401 pad 2: Net-(C401-Pad2) -> GND
- SW401 pad 3: /VCA_ENV -> Net-(C403-Pad2)
- U201 pad 2: Net-(C201-Pad1) -> /modulation_ADSR/OUT
- U201 pad 3: GND -> Net-(C202-Pad1)
- U201 pad 5: GND -> Net-(RV203-Pad2)
- U201 pad 6: Net-(C203-Pad1) -> Net-(RV202-Pad2)
- U201 pad 7: Net-(C203-Pad2) -> Net-(RV202-Pad2)
- U202 pad 1: /modulation_ADSR/INVERTING_OUT -> GND
- U202 pad 2: Net-(R223-Pad2) -> Net-(Q203-Pad3)
- U202 pad 3: GND -> Net-(RV201-Pad1)
- U202 pad 4: -15V -> Net-(C201-Pad1)
- U202 pad 5: Net-(R231-Pad1) -> Net-(C204-Pad1)
- U202 pad 6: /MOD_ENV_GATE -> /modulation_ADSR/OUT
- U202 pad 7: Net-(D201-Pad2) -> Net-(Q201-Pad2)
- U301 pad 2: Net-(C301-Pad1) -> /VCF_ADSR/OUT
- U301 pad 3: GND -> Net-(C302-Pad1)
- U301 pad 5: GND -> Net-(RV303-Pad2)
- U301 pad 6: Net-(C303-Pad1) -> Net-(RV302-Pad2)
- U301 pad 7: Net-(C303-Pad2) -> Net-(RV302-Pad2)
- U302 pad 1: /VCF_ADSR/INVERTING_OUT -> GND
- U302 pad 2: Net-(R323-Pad2) -> Net-(Q303-Pad3)
- U302 pad 3: GND -> Net-(RV301-Pad1)
- U302 pad 4: -15V -> Net-(C301-Pad1)
- U302 pad 5: Net-(R331-Pad1) -> Net-(C304-Pad1)
- U302 pad 6: /VCF_ENV_GATE -> /VCF_ADSR/OUT
- U302 pad 7: Net-(D301-Pad2) -> Net-(Q301-Pad2)
- U401 pad 1: /VCA_ENV -> /VCA_ADSR/OUT
- U401 pad 2: Net-(C401-Pad1) -> /VCA_ADSR/OUT
- U401 pad 3: GND -> Net-(C402-Pad1)
- U401 pad 5: GND -> Net-(RV403-Pad2)
- U401 pad 6: Net-(C403-Pad1) -> Net-(RV402-Pad2)
- U401 pad 7: Net-(C403-Pad2) -> Net-(RV402-Pad2)
- U402 pad 1: /VCA_ADSR/INVERTING_OUT -> GND
- U402 pad 2: Net-(R423-Pad2) -> Net-(Q403-Pad3)
- U402 pad 3: GND -> Net-(RV401-Pad1)
- U402 pad 4: -15V -> Net-(C401-Pad1)
- U402 pad 5: Net-(R431-Pad1) -> Net-(C404-Pad1)
- U402 pad 6: /VCA_ENV_GATE -> /VCA_ADSR/OUT
- U402 pad 7: Net-(D401-Pad2) -> Net-(Q401-Pad2)
Routing:
- net +15V: track 304.9 -> 51.0 mm, vias 8 -> 0
- net -15V: track 178.6 -> 0.00 mm, vias 5 -> 0
- net Net-(Q202-Pad1): track 156.3 -> 14.8 mm, vias 2 -> 0
- net Net-(D202-Pad2): track 0.00 -> 137.8 mm, vias 0 -> 2
- net Net-(Q207-Pad3): track 107.3 -> 0.00 mm, vias 2 -> 0
- net Net-(D202-Pad1): track 100.8 -> 0.00 mm, vias 2 -> 0
- net Net-(Q201-Pad2): track 105.2 -> 7.28 mm, vias 3 -> 0
- net Net-(C201-Pad1): track 53.4 -> 143.2 mm, vias 2 -> 3
- net Net-(D204-Pad2): track 85.6 -> 0.00 mm, vias 2 -> 0
- net Net-(D201-Pad1): track 23.5 -> 104.7 mm, vias 0 -> 2
- net Net-(RV201-Pad1): track 0.00 -> 80.6 mm
- net Net-(RV202-Pad2): track 0.00 -> 78.6 mm, vias 0 -> 3
- net Net-(C202-Pad1): track 0.00 -> 65.1 mm
- net Net-(C203-Pad1): track 51.7 -> 0.00 mm, vias 2 -> 0
- net /modulation_ADSR/OUT: track 111.3 -> 70.8 mm, vias 1 -> 4
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Other:
- board size 175.3 x 111.8 mm -> 172.7 x 107.9 mm

Commit message: Progress on ADSR layout
Parts:
- removed R103, R105: 100k, Resistor_SMD:R_0805_2012Metric
- removed R104, R106, R107: 1k, Resistor_SMD:R_0805_2012Metric
- added TP1: mod env gate, TestPoint:TestPoint_Keystone_5000-5004_Miniature, B.Cu at (156.2, 47.6)
- added TP2: VCF env gate, TestPoint:TestPoint_Keystone_5000-5004_Miniature, B.Cu at (156.2, 92.1)
- added TP3: VCA env gate, TestPoint:TestPoint_Keystone_5000-5004_Miniature, B.Cu at (111.1, 92.1)
- added TP4: mod env, TestPoint:TestPoint_Keystone_5000-5004_Miniature, B.Cu at (120.7, 47.6)
- added TP5: inv mod env, TestPoint:TestPoint_Keystone_5000-5004_Miniature, B.Cu at (120.7, 58.7)
- added TP6: VCF env, TestPoint:TestPoint_Keystone_5000-5004_Miniature, B.Cu at (120.7, 92.1)
- added TP7: VCA env, TestPoint:TestPoint_Keystone_5000-5004_Miniature, B.Cu at (76.8, 92.1)
- R101, R102: value 1k -> 100k
- moved R307 213.4 mm to (27.9, 73.2), turned to 0 degrees
- moved R407 211.2 mm to (27.9, 116.8), turned to 0 degrees
- moved U402 206.5 mm to (91.9, 72.9)
- moved D402 203.1 mm to (82.9, 89.4)
- moved D401 199.2 mm to (82.9, 81.3), turned to 0 degrees
- moved D403 199.0 mm to (82.9, 85.3), turned to 0 degrees
- moved Q401 193.4 mm to (82.9, 72.4)
- moved D405 183.1 mm to (106.8, 79.5), turned to 0 degrees
- moved C401 180.6 mm to (100.5, 79.8)
- moved Q402 175.7 mm to (100.5, 87.9)
- moved C402 174.1 mm to (85.6, 95.8)
- moved R406 169.6 mm to (100.5, 67.6)
- moved R303 168.9 mm to (72.4, 73.2), turned to 0 degrees
- moved R405 167.7 mm to (100.5, 83.3), turned to 0 degrees
- moved R403 167.4 mm to (72.1, 116.8), turned to 0 degrees
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Connections:
- J2 pad 1: Net-(J2-Pad1) -> /modulation_ADSR/OUT
- J3 pad 1: Net-(J3-Pad1) -> /modulation_ADSR/OUT
- J3 pad 2: Net-(J3-Pad2) -> Net-(R102-Pad2)
- J4 pad 1: Net-(J4-Pad1) -> /VCF_ADSR/OUT
- R101 pad 2: Net-(J2-Pad1) -> Net-(R102-Pad1)
- R102 pad 1: /modulation_ADSR/OUT -> Net-(R102-Pad1)
- R102 pad 2: Net-(J3-Pad1) -> Net-(R102-Pad2)
- U101 pad 1: Net-(R103-Pad2) -> Net-(U101-Pad1)
- U101 pad 2: Net-(R103-Pad1) -> Net-(U101-Pad1)
- U101 pad 6: Net-(U101-Pad6) -> Net-(R102-Pad1)
- U101 pad 7: Net-(U101-Pad6) -> Net-(R102-Pad2)
- U201 pad 1: /modulation_ADSR/OUT -> Net-(RV202-Pad2)
- U201 pad 2: /modulation_ADSR/OUT -> Net-(RV202-Pad2)
- U201 pad 3: Net-(C202-Pad1) -> Net-(RV203-Pad2)
- U201 pad 5: Net-(RV203-Pad2) -> Net-(C202-Pad1)
- U201 pad 6: Net-(RV202-Pad2) -> /modulation_ADSR/OUT
- U201 pad 7: Net-(RV202-Pad2) -> /modulation_ADSR/OUT
- U301 pad 1: /VCF_ADSR/OUT -> Net-(RV302-Pad2)
- U301 pad 2: /VCF_ADSR/OUT -> Net-(RV302-Pad2)
- U301 pad 3: Net-(C302-Pad1) -> Net-(RV303-Pad2)
- U301 pad 5: Net-(RV303-Pad2) -> Net-(C302-Pad1)
- U301 pad 6: Net-(RV302-Pad2) -> /VCF_ADSR/OUT
- U301 pad 7: Net-(RV302-Pad2) -> /VCF_ADSR/OUT
- U401 pad 1: /VCA_ADSR/OUT -> Net-(RV402-Pad2)
- U401 pad 2: /VCA_ADSR/OUT -> Net-(RV402-Pad2)
- U401 pad 3: Net-(C402-Pad1) -> Net-(RV403-Pad2)
- U401 pad 5: Net-(RV403-Pad2) -> Net-(C402-Pad1)
- U401 pad 6: Net-(RV402-Pad2) -> /VCA_ENV
- U401 pad 7: Net-(RV402-Pad2) -> /VCA_ENV
- U402 pad 6: /VCA_ADSR/OUT -> /VCA_ENV
Routing:
- net +15V: track 51.0 -> 407.2 mm, vias 0 -> 2
- net /modulation_ADSR/GATE: track 0.00 -> 170.4 mm
- net -15V: track 0.00 -> 139.2 mm
- net /modulation_ADSR/OUT: track 70.8 -> 207.7 mm, vias 4 -> 3
- net /VCF_ADSR/OUT: track 0.00 -> 135.3 mm, vias 0 -> 1
- net Net-(C401-Pad1): track 0.00 -> 132.8 mm, vias 0 -> 2
- net Net-(C402-Pad1): track 0.00 -> 127.0 mm, vias 0 -> 1
- net Net-(RV301-Pad1): track 0.00 -> 126.1 mm, vias 0 -> 1
- net Net-(RV401-Pad1): track 0.00 -> 118.1 mm, vias 0 -> 2
- net Net-(D403-Pad1): track 0.00 -> 112.6 mm, vias 0 -> 2
- net Net-(D302-Pad2): track 0.00 -> 106.9 mm, vias 0 -> 2
- net Net-(R102-Pad2): track 0.00 -> 106.8 mm
- net /VCF_ADSR/GATE: track 0.00 -> 102.0 mm, vias 0 -> 1
- net Net-(C302-Pad1): track 0.00 -> 90.7 mm, vias 0 -> 1
- net Net-(C201-Pad1): track 143.2 -> 56.9 mm, vias 3 -> 0
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Other:
- board text added: "ADSR board rev 0 2022-06-12"
- board text added: "DC POWER IN"
- board text added: "GND"
- board text added: "MODOSC BOARD PORT"
- board text added: "Ox Ribbon Synth"
- board text added: "RIBBON BOARD PORT"
- board text added: "V+"
- board text added: "V-"
- board text added: "VCA env"
- board text added: "VCA env gate"
- board text added: "VCF BOARD PORT"
- board text added: "VCF env"
- board text added: "VCF env gate"
- board text added: "VCO BOARD PORT"
- board text added: "inv mod env"
- board text added: "mod env"
- board text added: "mod env gate"

Commit message: Move some headers for better alignment
Parts:
- moved J2 34.9 mm to (83.2, 116.2)
- moved J4 19.7 mm to (27.9, 104.1)
- moved J1 9.52 mm to (98.4, 116.2)
- moved TP501 3.19 mm to (90.2, 98.4)
- moved TP503 2.99 mm to (95.9, 98.4)
- moved J3 0.63 mm to (28.0, 57.1)
Routing:
- net /modulation_ADSR/OUT: track 207.7 -> 236.3 mm
- net /VCF_ADSR/OUT: track 135.3 -> 150.8 mm
- net /VCA_ADSR/GATE: track 44.8 -> 29.5 mm, vias 1 -> 0
- net /modulation_ADSR/GATE: track 170.4 -> 157.1 mm
- net /VCF_ADSR/GATE: track 102.0 -> 92.7 mm
- net /VCA_ENV: track 83.2 -> 92.4 mm
- net +15V: track 407.2 -> 404.4 mm
- net -15V: track 139.2 -> 136.8 mm
- net Net-(C402-Pad1): track 127.0 -> 127.9 mm
- net Net-(R102-Pad2): track 106.8 -> 107.5 mm
- net GND: vias 33 -> 32
Other:
- board text added: "INV MOD ENV O"
- board text added: "MOD ENV I"
- board text added: "MOD ENV O"
- board text added: "VCA ENV I"
- board text added: "VCA ENV O"
- board text added: "VCF ENV I"
- board text added: "VCF ENV O"
