File: summer_2022_refurb/ribbon_board/clocked_s_and_h.kicad_sch (KiCad schematic)
At the start: 12 parts

Commit message: Ribbon board progress, tidy up schem
Other:
- title: (none) -> Josh Ox Ribbon Synth Ribbon board
Changed lines of the file:
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@@
 (kicad_sch (version 20211123) (generator eeschema)
   (paper "A4")
+  (title_block
+    (title "Josh Ox Ribbon Synth Ribbon board")
+    (date "2022-06-16")
+    (rev "0")
+    (comment 1 "creativecommons.org/licences/by/4.0")
+    (comment 2 "license: CC by 4.0")
+    (comment 3 "Author: Jordan Aceto")
+  )
   (junction (at 160.02 130.81) (diameter 0) (color 0 0 0 0)
   )
