File: summer_2022_refurb/ribbon_board/gate_controller.kicad_sch (KiCad schematic)
At the start: 6 parts

Commit message: Ribbon board progress, tidy up schem
Connections:
- net +15V: now also R?.2; no longer R?.1
- net GND: now also R?.1; no longer R?.2
- net VCA_ADSR_gate_logic/IN_A renamed VCA_ADSR_gate_logic/RIBBON_GATE
- net VCA_ADSR_gate_logic/IN_B renamed VCA_ADSR_gate_logic/AUTO_GATE
Other:
- sheet VCA_ADSR_gate_logic ports: added AUTO_GATE, RIBBON_GATE; removed IN_A, IN_B
- sheet VCF_ADSR_gate_logic ports: added AUTO_GATE, RIBBON_GATE; removed IN_A, IN_B
- sheet mod_ADSR_gate_logic ports: added AUTO_GATE, RIBBON_GATE; removed IN_A, IN_B
- sheet s&h_gate_logic3 ports: added AUTO_GATE, RIBBON_GATE; removed IN_A, IN_B
- title: (none) -> Josh Ox Ribbon Synth Ribbon board
- moved on the sheet: R?, SW?, U?B
