File: summer_2022_refurb/ribbon_board/gate_logic.kicad_sch (KiCad schematic)
At the start: 8 parts

Commit message: Ribbon board progress, tidy up schem
Connections:
- net at SW?.1: now also D?.2 (A); no longer D?.2 (A)
- net at SW?.3: now also D?.2 (A); no longer D?.2 (A)
- net IN_A renamed RIBBON_GATE
- net IN_B renamed AUTO_GATE
Other:
- note added: "Gate mode switch 1) ribbon (ext) 2) both (AND) 3) auto gate"
- title: (none) -> Josh Ox Ribbon Synth Ribbon board
Changed lines of the file:
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@@
 (kicad_sch (version 20211123) (generator eeschema)
   (paper "A4")
+  (title_block
+    (title "Josh Ox Ribbon Synth Ribbon board")
+    (date "2022-06-16")
+    (rev "0")
+    (comment 1 "creativecommons.org/licences/by/4.0")
+    (comment 2 "license: CC by 4.0")
+    (comment 3 "Author: Jordan Aceto")
+  )
   (junction (at 144.78 105.41) (diameter 0) (color 0 0 0 0)
   )
@@
     (stroke (width 0) (type default) (color 0 0 0 0))
   )
-  (hierarchical_label "IN_B" (shape input) (at 100.33 121.92 180)
+  (text "Gate mode switch\n\n1) ribbon (ext)\n2) both (AND)\n3) auto gate"
+    (at 81.28 97.79 0)
+    (effects (font (size 1.27 1.27)) (justify left bottom))
+  )
+  (hierarchical_label "AUTO_GATE" (shape input) (at 100.33 121.92 180)
     (effects (font (size 1.27 1.27)) (justify right))
   )
@@
     (effects (font (size 1.27 1.27)) (justify left))
   )
-  (hierarchical_label "IN_A" (shape input) (at 100.33 67.31 180)
+  (hierarchical_label "RIBBON_GATE" (shape input) (at 100.33 67.31 180)
     (effects (font (size 1.27 1.27)) (justify right))
   )
@@
     (pin "2")
   )
-  (symbol (lib_id "Switch:SW_SPDT_MSM") (at 118.11 95.25 0) (unit 1)
+  (symbol (lib_id "Switch:SW_SPDT_MSM") (at 118.11 95.25 0) (mirror x) (unit 1)
     (in_bom yes) (on_board yes) (fields_autoplaced)
     (property "Reference" "SW?" (id 0) (at 118.237 87.63 0))
