File: summer_2022_refurb/VCF_VCA_board/kicad_6_docs/VCA.kicad_sch (KiCad schematic)
At the start: 22 parts, among them U10 SSI2164, U11 SSI2164, U6 TL072, U7 TL072

Commit message: Change directory structure, minor schem and pcb tweaks
Parts:
- renumbered C601 to C401, C602 to C402, C603 to C403, C604 to C404, C605 to C405, D601 to D401, D602 to D402, R601 to R401, R602 to R402, R603 to R403, R604 to R404, R605 to R405, R606 to R406, R607 to R407, R608 to R408, R609 to R409, R610 to R410, R611 to R411
Changed lines of the file:
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@@
   (symbol (lib_id "Device:R") (at 135.89 69.85 90) (unit 1)
     (in_bom yes) (on_board yes) (fields_autoplaced)
-    (property "Reference" "R603" (id 0) (at 135.89 63.5 90))
+    (property "Reference" "R403" (id 0) (at 135.89 63.5 90))
     (property "Value" "30k" (id 1) (at 135.89 66.04 90))
     (property "Footprint" "Resistor_SMD:R_0805_2012Metric" (id 2) (at 135.89 71.628 90)
@@
   (symbol (lib_id "Device:C") (at 125.73 132.08 0) (mirror y) (unit 1)
     (in_bom yes) (on_board yes) (fields_autoplaced)
-    (property "Reference" "C604" (id 0) (at 129.54 130.8099 0)
+    (property "Reference" "C404" (id 0) (at 129.54 130.8099 0)
       (effects (font (size 1.27 1.27)) (justify right))
     )
@@
   (symbol (lib_id "Device:R") (at 85.09 115.57 90) (unit 1)
     (in_bom yes) (on_board yes)
-    (property "Reference" "R607" (id 0) (at 85.09 110.49 90))
+    (property "Reference" "R407" (id 0) (at 85.09 110.49 90))
     (property "Value" "10M" (id 1) (at 85.09 113.03 90))
     (property "Footprint" "Resistor_SMD:R_0805_2012Metric" (id 2) (at 85.09 117.348 90)
@@
   (symbol (lib_id "Device:C") (at 181.61 48.26 90) (unit 1)
     (in_bom yes) (on_board yes) (fields_autoplaced)
-    (property "Reference" "C601" (id 0) (at 181.61 40.64 90))
+    (property "Reference" "C401" (id 0) (at 181.61 40.64 90))
     (property "Value" "100p" (id 1) (at 181.61 43.18 90))
     (property "Footprint" "Capacitor_SMD:C_0805_2012Metric" (id 2) (at 185.42 47.2948 0)
@@
   (symbol (lib_id "Device:C") (at 101.6 146.05 90) (unit 1)
     (in_bom yes) (on_board yes) (fields_autoplaced)
-    (property "Reference" "C605" (id 0) (at 101.6 138.43 90))
+    (property "Reference" "C405" (id 0) (at 101.6 138.43 90))
     (property "Value" "100p" (id 1) (at 101.6 140.97 90))
     (property "Footprint" "Capacitor_SMD:C_0805_2012Metric" (id 2) (at 105.41 145.0848 0)
@@
   (symbol (lib_id "Device:R") (at 144.78 78.74 0) (mirror y) (unit 1)
     (in_bom yes) (on_board yes) (fields_autoplaced)
-    (property "Reference" "R605" (id 0) (at 147.32 77.4699 0)
+    (property "Reference" "R405" (id 0) (at 147.32 77.4699 0)
       (effects (font (size 1.27 1.27)) (justify right))
     )
@@
   (symbol (lib_id "Device:R") (at 181.61 60.96 90) (unit 1)
     (in_bom yes) (on_board yes) (fields_autoplaced)
-    (property "Reference" "R602" (id 0) (at 181.61 54.61 90))
+    (property "Reference" "R402" (id 0) (at 181.61 54.61 90))
     (property "Value" "30k" (id 1) (at 181.61 57.15 90))
     (property "Footprint" "Resistor_SMD:R_0805_2012Metric" (id 2) (at 181.61 62.738 90)
@@
   (symbol (lib_id "Device:R") (at 125.73 121.92 0) (mirror y) (unit 1)
     (in_bom yes) (on_board yes) (fields_autoplaced)
-    (property "Reference" "R609" (id 0) (at 128.27 120.6499 0)
+    (property "Reference" "R409" (id 0) (at 128.27 120.6499 0)
       (effects (font (size 1.27 1.27)) (justify right))
     )
@@
   (symbol (lib_id "Device:R") (at 125.73 157.48 90) (unit 1)
     (in_bom yes) (on_board yes)
-    (property "Reference" "R611" (id 0) (at 125.73 151.13 90))
+    (property "Reference" "R411" (id 0) (at 125.73 151.13 90))
     (property "Value" "4k7" (id 1) (at 125.73 153.67 90))
     (property "Footprint" "Resistor_SMD:R_0805_2012Metric" (id 2) (at 125.73 159.258 90)
@@
   (symbol (lib_id "Device:R") (at 198.12 72.39 90) (unit 1)
     (in_bom yes) (on_board yes) (fields_autoplaced)
-    (property "Reference" "R604" (id 0) (at 198.12 66.04 90))
+    (property "Reference" "R404" (id 0) (at 198.12 66.04 90))
     (property "Value" "1k" (id 1) (at 198.12 68.58 90))
     (property "Footprint" "Resistor_SMD:R_0805_2012Metric" (id 2) (at 198.12 74.168 90)
@@
   (symbol (lib_id "Device:R") (at 224.79 85.09 0) (unit 1)
     (in_bom yes) (on_board yes) (fields_autoplaced)
-    (property "Reference" "R606" (id 0) (at 227.33 83.8199 0)
+    (property "Reference" "R406" (id 0) (at 227.33 83.8199 0)
       (effects (font (size 1.27 1.27)) (justify left))
     )
@@
   (symbol (lib_id "Device:R") (at 132.08 115.57 270) (mirror x) (unit 1)
     (in_bom yes) (on_board yes)
-    (property "Reference" "R608" (id 0) (at 132.08 110.49 90))
+    (property "Reference" "R408" (id 0) (at 132.08 110.49 90))
     (property "Value" "100k" (id 1) (at 132.08 113.03 90))
     (property "Footprint" "Resistor_SMD:R_0805_2012Metric" (id 2) (at 132.08 117.348 90)
@@
   (symbol (lib_id "Device:R") (at 85.09 154.94 90) (unit 1)
     (in_bom yes) (on_board yes) (fields_autoplaced)
-    (property "Reference" "R610" (id 0) (at 85.09 148.59 90))
+    (property "Reference" "R410" (id 0) (at 85.09 148.59 90))
     (property "Value" "100k" (id 1) (at 85.09 151.13 90))
     (property "Footprint" "Resistor_SMD:R_0805_2012Metric" (id 2) (at 85.09 156.718 90)
@@
   (symbol (lib_id "Device:C") (at 217.17 72.39 90) (unit 1)
     (in_bom yes) (on_board yes) (fields_autoplaced)
-    (property "Reference" "C602" (id 0) (at 217.17 64.77 90))
+    (property "Reference" "C402" (id 0) (at 217.17 64.77 90))
     (property "Value" "10u" (id 1) (at 217.17 67.31 90))
     (property "Footprint" "Capacitor_THT:C_Radial_D6.3mm_H5.0mm_P2.50mm" (id 2) (at 220.98 71.4248 0)
@@
   (symbol (lib_id "Device:R") (at 135.89 58.42 90) (unit 1)
     (in_bom yes) (on_board yes) (fields_autoplaced)
-    (property "Reference" "R601" (id 0) (at 135.89 52.07 90))
+    (property "Reference" "R401" (id 0) (at 135.89 52.07 90))
     (property "Value" "30k" (id 1) (at 135.89 54.61 90))
     (property "Footprint" "Resistor_SMD:R_0805_2012Metric" (id 2) (at 135.89 60.198 90)
@@
   (symbol (lib_id "Device:C") (at 144.78 88.9 0) (mirror y) (unit 1)
     (in_bom yes) (on_board yes) (fields_autoplaced)
-    (property "Reference" "C603" (id 0) (at 148.59 87.6299 0)
+    (property "Reference" "C403" (id 0) (at 148.59 87.6299 0)
       (effects (font (size 1.27 1.27)) (justify right))
     )
@@
   (symbol (lib_id "Device:D_Zener") (at 207.01 90.17 90) (unit 1)
     (in_bom yes) (on_board yes) (fields_autoplaced)
-    (property "Reference" "D602" (id 0) (at 209.55 88.8999 90)
+    (property "Reference" "D402" (id 0) (at 209.55 88.8999 90)
       (effects (font (size 1.27 1.27)) (justify right))
     )
@@
   (symbol (lib_id "Device:D_Zener") (at 207.01 80.01 270) (unit 1)
     (in_bom yes) (on_board yes) (fields_autoplaced)
-    (property "Reference" "D601" (id 0) (at 209.55 78.7399 90)
+    (property "Reference" "D401" (id 0) (at 209.55 78.7399 90)
       (effects (font (size 1.27 1.27)) (justify left))
     )
