File: summer_2022_refurb/sample_and_hold_board/kicad_6_docs/power_supply.kicad_sch (KiCad schematic)
At the start: 17 parts, among them J4 power_entry, U1 TL072, U2 TL072, U3 TL072

Commit message: Change directory structure, minor schem and pcb tweaks
Parts:
- TP6, TP7, TP8: now left out of the parts list
Changed lines of the file:
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@@
   (title_block
     (title "Josh Ox Ribbon Synth Sample and Hold Board")
-    (date "2022-06-09")
+    (date "2022-06-16")
     (rev "0")
     (comment 1 "creativecommons.org/licences/by/4.0")
@@
   )
   (symbol (lib_id "Connector:TestPoint") (at 67.31 160.02 0) (unit 1)
-    (in_bom yes) (on_board yes) (fields_autoplaced)
+    (in_bom no) (on_board yes) (fields_autoplaced)
     (property "Reference" "TP7" (id 0) (at 69.85 155.4479 0)
       (effects (font (size 1.27 1.27)) (justify left))
@@
   )
   (symbol (lib_id "Connector:TestPoint") (at 62.23 173.99 180) (unit 1)
-    (in_bom yes) (on_board yes) (fields_autoplaced)
+    (in_bom no) (on_board yes) (fields_autoplaced)
     (property "Reference" "TP8" (id 0) (at 64.77 176.0219 0)
       (effects (font (size 1.27 1.27)) (justify right))
@@
   )
   (symbol (lib_id "Connector:TestPoint") (at 62.23 143.51 0) (unit 1)
-    (in_bom yes) (on_board yes) (fields_autoplaced)
+    (in_bom no) (on_board yes) (fields_autoplaced)
     (property "Reference" "TP6" (id 0) (at 64.77 138.9379 0)
       (effects (font (size 1.27 1.27)) (justify left))
