File: summer_2022_refurb/main_VCO_board/kicad_6_docs/audio_mixer.kicad_sch (KiCad schematic)
At the start: 14 parts

Commit message: Main VCO progress
Other:
- title: (none) -> Josh Ox Ribon Synth Main VCO board
- moved on the sheet: C?, R?, RV?, U?A

Commit message: Progress on main VCO, schem getting close but not done
Parts:
- added SW2201: SW_SPDT, symbol Switch:SW_SPDT
- added SW2202: SW_SPDT_CO, symbol Switch:SW_SPDT_MSM
- U18: renamed from U?; footprint (none) -> Package_SO:SOIC-8_3.9x4.9mm_P1.27mm
- gave numbers to parts that had none: 13
Connections:
- net MAIN_VCO: now also SW2201.1 (A); no longer RV2201.3
- net NOISE: no longer names the net of RV2205.3
- net NOISE: now also SW2202.2
- new net: RV2201.3, SW2201.2 (B)
- new net PINK_NOISE: SW2202.3
- new net WHITE_NOISE: SW2202.1
- no-connect marks 0 -> 1

Commit message: Remove white/pink noise switch from VCO, use the one on the S&H board
Parts:
- removed SW2202: SW_SPDT_CO, symbol Switch:SW_SPDT_MSM
- added SW2202: SW_SPDT, symbol Switch:SW_SPDT
Connections:
- net at RV2205.3: now also SW2202.2 (B)
- new net NOISE: SW2202.1 (A)
- no-connect marks 1 -> 2
Changed lines of the file:
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@@
   (junction (at 153.67 110.49) (diameter 0) (color 0 0 0 0)
   )
+  (no_connect (at 107.95 149.86))
   (no_connect (at 107.95 63.5))
   (wire (pts (xy 139.7 110.49) (xy 143.51 110.49))
@@
     (stroke (width 0) (type default) (color 0 0 0 0))
   )
-  (wire (pts (xy 105.41 149.86) (xy 107.95 149.86))
-    (stroke (width 0) (type default) (color 0 0 0 0))
-  )
   (wire (pts (xy 153.67 88.9) (xy 153.67 67.31))
     (stroke (width 0) (type default) (color 0 0 0 0))
@@
   (wire (pts (xy 151.13 132.08) (xy 153.67 132.08))
     (stroke (width 0) (type default) (color 0 0 0 0))
-  )
-  (hierarchical_label "PINK_NOISE" (shape input) (at 105.41 149.86 180)
-    (effects (font (size 1.27 1.27)) (justify right))
   )
   (hierarchical_label "OUT" (shape output) (at 191.77 99.06 0)
@@
     (effects (font (size 1.27 1.27)) (justify right))
   )
-  (hierarchical_label "WHITE_NOISE" (shape input) (at 105.41 144.78 180)
+  (hierarchical_label "NOISE" (shape input) (at 105.41 144.78 180)
     (effects (font (size 1.27 1.27)) (justify right))
   )
@@
     )
     (pin "1")
+  )
+  (symbol (lib_id "Switch:SW_SPDT") (at 113.03 147.32 0) (mirror y) (unit 1)
+    (in_bom yes) (on_board yes) (fields_autoplaced)
+    (property "Reference" "SW2202" (id 0) (at 113.03 139.7 0))
+    (property "Value" "SW_SPDT" (id 1) (at 113.03 142.24 0))
+    (property "Footprint" "" (id 2) (at 113.03 147.32 0)
+      (effects (font (size 1.27 1.27)) hide)
+    )
+    (property "Datasheet" "~" (id 3) (at 113.03 147.32 0)
+      (effects (font (size 1.27 1.27)) hide)
+    )
+    (pin "1")
+    (pin "2")
+    (pin "3")
   )
   (symbol (lib_id "power:GND") (at 135.89 138.43 0) (unit 1)
@@
     (pin "2")
   )
-  (symbol (lib_id "Switch:SW_SPDT_MSM") (at 113.03 147.32 0) (mirror y) (unit 1)
-    (in_bom yes) (on_board yes) (fields_autoplaced)
-    (property "Reference" "SW2202" (id 0) (at 112.903 139.7 0))
-    (property "Value" "SW_SPDT_CO" (id 1) (at 112.903 142.24 0))
-    (property "Footprint" "" (id 2) (at 113.03 147.32 0)
-      (effects (font (size 1.27 1.27)) hide)
-    )
-    (property "Datasheet" "~" (id 3) (at 113.03 147.32 0)
-      (effects (font (size 1.27 1.27)) hide)
-    )
-    (pin "1")
-    (pin "2")
-    (pin "3")
-  )
   (symbol (lib_id "Device:R") (at 147.32 88.9 90) (unit 1)

Commit message: Main VCO rough parts placement
Parts:
- C2201: footprint (none) -> Capacitor_SMD:C_0805_2012Metric
- R2201, R2202, R2203, R2204, R2205, R2206, R2207: footprint (none) -> Resistor_SMD:R_0805_2012Metric
- RV2201, RV2202, RV2203, RV2204, RV2205: footprint (none) -> Potentiometer_THT:Potentiometer_Alpha_RD901F-40-00D_Single_Vertical
- SW2201, SW2202: footprint (none) -> custom_footprints:SPDT_mini_toggle
Changed lines of the file:
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@@
     (property "Reference" "C2201" (id 0) (at 171.45 72.39 90))
     (property "Value" "10p" (id 1) (at 171.45 74.93 90))
-    (property "Footprint" "" (id 2) (at 175.26 79.0448 0)
+    (property "Footprint" "Capacitor_SMD:C_0805_2012Metric" (id 2) (at 175.26 79.0448 0)
       (effects (font (size 1.27 1.27)) hide)
     )
@@
       (effects (font (size 1.27 1.27)) (justify right))
     )
-    (property "Footprint" "" (id 2) (at 135.89 110.49 0)
+    (property "Footprint" "Potentiometer_THT:Potentiometer_Alpha_RD901F-40-00D_Single_Vertical" (id 2) (at 135.89 110.49 0)
       (effects (font (size 1.27 1.27)) hide)
     )
@@
       (effects (font (size 1.27 1.27)) (justify right))
     )
-    (property "Footprint" "" (id 2) (at 135.89 153.67 0)
+    (property "Footprint" "Potentiometer_THT:Potentiometer_Alpha_RD901F-40-00D_Single_Vertical" (id 2) (at 135.89 153.67 0)
       (effects (font (size 1.27 1.27)) hide)
     )
@@
     (property "Reference" "R2204" (id 0) (at 147.32 104.14 90))
     (property "Value" "100k" (id 1) (at 147.32 106.68 90))
-    (property "Footprint" "" (id 2) (at 147.32 112.268 90)
+    (property "Footprint" "Resistor_SMD:R_0805_2012Metric" (id 2) (at 147.32 112.268 90)
       (effects (font (size 1.27 1.27)) hide)
     )
@@
     (property "Reference" "SW2202" (id 0) (at 113.03 139.7 0))
     (property "Value" "SW_SPDT" (id 1) (at 113.03 142.24 0))
-    (property "Footprint" "" (id 2) (at 113.03 147.32 0)
+    (property "Footprint" "custom_footprints:SPDT_mini_toggle" (id 2) (at 113.03 147.32 0)
       (effects (font (size 1.27 1.27)) hide)
     )
@@
     (property "Reference" "R2205" (id 0) (at 147.32 125.73 90))
     (property "Value" "100k" (id 1) (at 147.32 128.27 90))
-    (property "Footprint" "" (id 2) (at 147.32 133.858 90)
+    (property "Footprint" "Resistor_SMD:R_0805_2012Metric" (id 2) (at 147.32 133.858 90)
       (effects (font (size 1.27 1.27)) hide)
     )
@@
       (effects (font (size 1.27 1.27)) (justify right))
     )
-    (property "Footprint" "" (id 2) (at 135.89 132.08 0)
+    (property "Footprint" "Potentiometer_THT:Potentiometer_Alpha_RD901F-40-00D_Single_Vertical" (id 2) (at 135.89 132.08 0)
       (effects (font (size 1.27 1.27)) hide)
     )
@@
     (property "Reference" "R2202" (id 0) (at 147.32 60.96 90))
     (property "Value" "100k" (id 1) (at 147.32 63.5 90))
-    (property "Footprint" "" (id 2) (at 147.32 69.088 90)
+    (property "Footprint" "Resistor_SMD:R_0805_2012Metric" (id 2) (at 147.32 69.088 90)
       (effects (font (size 1.27 1.27)) hide)
     )
@@
     (property "Reference" "R2201" (id 0) (at 147.32 39.37 90))
     (property "Value" "100k" (id 1) (at 147.32 41.91 90))
-    (property "Footprint" "" (id 2) (at 147.32 47.498 90)
+    (property "Footprint" "Resistor_SMD:R_0805_2012Metric" (id 2) (at 147.32 47.498 90)
       (effects (font (size 1.27 1.27)) hide)
     )
@@
     (property "Reference" "SW2201" (id 0) (at 113.03 53.34 0))
     (property "Value" "SW_SPDT" (id 1) (at 113.03 55.88 0))
-    (property "Footprint" "" (id 2) (at 113.03 60.96 0)
+    (property "Footprint" "custom_footprints:SPDT_mini_toggle" (id 2) (at 113.03 60.96 0)
       (effects (font (size 1.27 1.27)) hide)
     )
@@
     (property "Reference" "R2206" (id 0) (at 147.32 147.32 90))
     (property "Value" "100k" (id 1) (at 147.32 149.86 90))
-    (property "Footprint" "" (id 2) (at 147.32 155.448 90)
+    (property "Footprint" "Resistor_SMD:R_0805_2012Metric" (id 2) (at 147.32 155.448 90)
       (effects (font (size 1.27 1.27)) hide)
     )
@@
       (effects (font (size 1.27 1.27)) (justify right))
     )
-    (property "Footprint" "" (id 2) (at 135.89 88.9 0)
+    (property "Footprint" "Potentiometer_THT:Potentiometer_Alpha_RD901F-40-00D_Single_Vertical" (id 2) (at 135.89 88.9 0)
       (effects (font (size 1.27 1.27)) hide)
     )
@@
       (effects (font (size 1.27 1.27)) (justify right))
     )
-    (property "Footprint" "" (id 2) (at 135.89 67.31 0)
+    (property "Footprint" "Potentiometer_THT:Potentiometer_Alpha_RD901F-40-00D_Single_Vertical" (id 2) (at 135.89 67.31 0)
       (effects (font (size 1.27 1.27)) hide)
     )
@@
     (property "Reference" "R2207" (id 0) (at 171.45 85.09 90))
     (property "Value" "82k" (id 1) (at 171.45 87.63 90))
-    (property "Footprint" "" (id 2) (at 171.45 93.218 90)
+    (property "Footprint" "Resistor_SMD:R_0805_2012Metric" (id 2) (at 171.45 93.218 90)
       (effects (font (size 1.27 1.27)) hide)
     )
@@
     (property "Reference" "R2203" (id 0) (at 147.32 82.55 90))
     (property "Value" "100k" (id 1) (at 147.32 85.09 90))
-    (property "Footprint" "" (id 2) (at 147.32 90.678 90)
-      (effects (font (size 1.27 1.27)) hide)
-    )
+    (property "Footprint" "Resistor_SMD:R_0805_2012Metric" (id 2) (at 147.32 90.678 90)
+      (effects (font (size 1.27 1.27)) hide)
+    )
