File: summer_2022_refurb/main_VCO_board/kicad_6_docs/main_VCO_board.kicad_pcb (KiCad board)
At the start: 2 copper layers, 0 parts

Commit message: Main VCO rough parts placement
Parts:
- added C1001: C, Capacitor_SMD:C_0805_2012Metric, B.Cu at (55.2, 104.8)
- added C1101: C, Capacitor_SMD:C_0805_2012Metric, B.Cu at (70.5, 104.8)
- added C1201: 10p, Capacitor_SMD:C_0805_2012Metric, B.Cu at (70.5, 120.0)
- added C1401: 220n, Capacitor_THT:C_Rect_L7.0mm_W2.5mm_P5.00mm, B.Cu at (147.9, 94.0)
- added C1501: C, Capacitor_SMD:C_0805_2012Metric, B.Cu at (71.1, 68.6)
- added C1601: 10u, Capacitor_SMD:C_0805_2012Metric, B.Cu at (81.3, 13.3)
- added C1602: 10u BP, Capacitor_THT:C_Radial_D6.3mm_H5.0mm_P2.50mm, B.Cu at (80.0, 19.7)
- added C1603: 100p, Capacitor_SMD:C_0805_2012Metric, B.Cu at (61.0, 28.6)
- added C1701: C, Capacitor_SMD:C_0805_2012Metric, B.Cu at (71.1, 53.3)
- added C1801: C, Capacitor_SMD:C_0805_2012Metric, B.Cu at (54.6, 53.3)
- added C1901: C, Capacitor_SMD:C_0805_2012Metric, B.Cu at (103.5, 27.9)
- added C2001: 10p, Capacitor_SMD:C_0805_2012Metric, B.Cu at (149.2, 40.0)
- added C2002: 10p, Capacitor_SMD:C_0805_2012Metric, B.Cu at (149.2, 28.6)
- added C2003: 100p, Capacitor_SMD:C_0805_2012Metric, B.Cu at (149.2, 24.8)
- added C2004: 100p, Capacitor_SMD:C_0805_2012Metric, B.Cu at (149.2, 13.3)
- added C2005: 10p, Capacitor_SMD:C_0805_2012Metric, B.Cu at (134.0, 24.8)
- added C2006: 10p, Capacitor_SMD:C_0805_2012Metric, B.Cu at (134.0, 13.3)
- added C201: C, Capacitor_SMD:C_0805_2012Metric, B.Cu at (167.0, 162.6)
- added C202: 220n, Capacitor_THT:C_Rect_L7.0mm_W2.5mm_P5.00mm, B.Cu at (144.1, -8.26)
- added C2101: 100p, Capacitor_SMD:C_0805_2012Metric, B.Cu at (170.8, 48.7)
- added C2102: 100p, Capacitor_SMD:C_0805_2012Metric, B.Cu at (155.6, 48.7)
- added C2103: 100p, Capacitor_SMD:C_0805_2012Metric, B.Cu at (88.3, 33.0)
- added C2104: 100p, Capacitor_SMD:C_0805_2012Metric, B.Cu at (88.3, 21.6)
- added C2201: 10p, Capacitor_SMD:C_0805_2012Metric, B.Cu at (188.6, 93.3)
- added C2301: 100n, Capacitor_SMD:C_0805_2012Metric, B.Cu at (177.1, 181.6)
- added C2302: 100n, Capacitor_SMD:C_0805_2012Metric, B.Cu at (172.0, 181.6)
- added C2303: 100n, Capacitor_SMD:C_0805_2012Metric, B.Cu at (148.5, 141.6)
- added C2304: 100n, Capacitor_SMD:C_0805_2012Metric, B.Cu at (143.4, 141.6)
- added C2305: 100n, Capacitor_SMD:C_0805_2012Metric, B.Cu at (125.8, 77.5)
- added C2306: 100n, Capacitor_SMD:C_0805_2012Metric, B.Cu at (120.7, 77.5)
- added C2307: 100n, Capacitor_SMD:C_0805_2012Metric, B.Cu at (65.4, 120.0)
- added C2308: 100n, Capacitor_SMD:C_0805_2012Metric, B.Cu at (60.3, 120.0)
- added C2309: 100n, Capacitor_SMD:C_0805_2012Metric, B.Cu at (65.4, 68.6)
- added C2310: 100n, Capacitor_SMD:C_0805_2012Metric, B.Cu at (60.3, 68.6)
- added C2311: 10u, Capacitor_THT:CP_Radial_D6.3mm_P2.50mm, B.Cu at (137.2, 173.9)
- added C2312: 10u, Capacitor_THT:CP_Radial_D6.3mm_P2.50mm, B.Cu at (129.5, 173.9)
- added C2313: 100n, Capacitor_SMD:C_0805_2012Metric, B.Cu at (71.1, 18.4)
- added C2314: 100n, Capacitor_SMD:C_0805_2012Metric, B.Cu at (66.0, 18.4)
- added C2315: 100n, Capacitor_SMD:C_0805_2012Metric, B.Cu at (98.4, 35.6)
- added C2316: 100n, Capacitor_SMD:C_0805_2012Metric, B.Cu at (93.3, 35.6)
- added C2317: 100n, Capacitor_SMD:C_0805_2012Metric, B.Cu at (144.1, 41.9)
- added C2318: 100n, Capacitor_SMD:C_0805_2012Metric, B.Cu at (139.1, 41.9)
- added C2319: 330n, Capacitor_SMD:C_0805_2012Metric, B.Cu at (115.2, 177.8)
- added C2320: 330n, Capacitor_SMD:C_0805_2012Metric, B.Cu at (115.1, 184.8)
- added C2321: 100n, Capacitor_SMD:C_0805_2012Metric, B.Cu at (144.1, 24.8)
- added C2322: 100n, Capacitor_SMD:C_0805_2012Metric, B.Cu at (139.1, 24.8)
- added C2323: 100n, Capacitor_SMD:C_0805_2012Metric, B.Cu at (160.5, 56.4)
- added C2324: 100n, Capacitor_SMD:C_0805_2012Metric, B.Cu at (165.5, 56.4)
- added C2325: 100n, Capacitor_SMD:C_0805_2012Metric, B.Cu at (115.2, 174.0)
- added C2326: 100n, Capacitor_SMD:C_0805_2012Metric, B.Cu at (114.9, 188.6)
- added C2327: 100n, Capacitor_SMD:C_0805_2012Metric, B.Cu at (183.5, 104.8)
- added C2328: 100n, Capacitor_SMD:C_0805_2012Metric, B.Cu at (178.4, 104.8)
- added C2329: 100n, Capacitor_SMD:C_0805_2012Metric, B.Cu at (91.4, 122.6)
- added C2330: 100n, Capacitor_SMD:C_0805_2012Metric, B.Cu at (96.5, 132.1)
- added C2331: 100n, Capacitor_SMD:C_0805_2012Metric, B.Cu at (106.7, 143.5)
- added C2332: 100n, Capacitor_SMD:C_0805_2012Metric, B.Cu at (66.4, 29.2)
- added C2333: 100n, Capacitor_SMD:C_0805_2012Metric, B.Cu at (173.4, 108.6)
- added C2334: 100n, Capacitor_SMD:C_0805_2012Metric, B.Cu at (48.9, 141.0)
- added C2335: 100n, Capacitor_SMD:C_0805_2012Metric, B.Cu at (61.0, 37.5)
- added C2336: 100n, Capacitor_SMD:C_0805_2012Metric, B.Cu at (143.8, 154.9)
- added C2337: 100n, Capacitor_SMD:C_0805_2012Metric, B.Cu at (58.4, 131.4)
- added C2338: 100n, Capacitor_SMD:C_0805_2012Metric, B.Cu at (173.4, 93.3)
- added C2339: 100n, Capacitor_SMD:C_0805_2012Metric, B.Cu at (120.7, 88.3)
- added C2340: 100n, Capacitor_SMD:C_0805_2012Metric, B.Cu at (71.8, 163.8)
- added C2341: 100n, Capacitor_SMD:C_0805_2012Metric, B.Cu at (43.2, 132.7)
- added C2342: 100n, Capacitor_SMD:C_0805_2012Metric, B.Cu at (67.9, 168.3)
- added C301: 10u, Capacitor_SMD:C_0805_2012Metric, B.Cu at (86.4, 135.9)
- added C302: 10N, Capacitor_SMD:C_0805_2012Metric, B.Cu at (86.4, 132.1)
- added C303: 3N9 COG, Capacitor_SMD:C_0805_2012Metric, B.Cu at (96.5, 143.5)
- added C401: 100n, Capacitor_THT:C_Rect_L7.0mm_W2.5mm_P5.00mm, B.Cu at (138.4, 125.7)
- added C402: 20p, Capacitor_SMD:C_0805_2012Metric, B.Cu at (138.4, 130.2)
- added C403: 100p, Capacitor_SMD:C_0805_2012Metric, B.Cu at (138.4, 153.0)
- added C404: 100p, Capacitor_SMD:C_0805_2012Metric, B.Cu at (138.4, 141.6)
- added C501: 220n, Capacitor_THT:C_Rect_L7.0mm_W2.5mm_P5.00mm, B.Cu at (181.6, 178.4)
- added C502: 100p, Capacitor_SMD:C_0805_2012Metric, B.Cu at (166.9, 181.6)
- added C601: 220n, Capacitor_THT:C_Rect_L7.0mm_W2.5mm_P5.00mm, B.Cu at (147.9, 63.5)
- added C701: C, Capacitor_SMD:C_0805_2012Metric, B.Cu at (153.7, 145.4)
- added C801: 10u, Capacitor_SMD:C_0805_2012Metric, B.Cu at (136.0, 72.4)
- added C802: 10u BP, Capacitor_THT:C_Radial_D6.3mm_H5.0mm_P2.50mm, B.Cu at (134.7, 78.7)
- added C803: 100p, Capacitor_SMD:C_0805_2012Metric, B.Cu at (115.7, 87.6)
- added C901: C, Capacitor_SMD:C_0805_2012Metric, B.Cu at (153.7, 130.2)
- added D1001: 1N4148W, Diode_SMD:D_SOD-123, B.Cu at (54.6, 112.4)
- added D1002: 1N4148W, Diode_SMD:D_SOD-123, B.Cu at (54.6, 116.2)
- added D1201: 5v1, Diode_SMD:D_SOD-123, B.Cu at (75.6, 127.6)
- added D1202: 5v1, Diode_SMD:D_SOD-123, B.Cu at (75.6, 123.8)
- added D1801: 1N4148W, Diode_SMD:D_SOD-123, B.Cu at (54.6, 61.0)
- added D1802: 1N4148W, Diode_SMD:D_SOD-123, B.Cu at (54.6, 64.8)
- added D2101: BAT48ZFILM, Diode_SMD:D_SOD-123, B.Cu at (180.3, 12.1)
- added D2102: BAT48ZFILM, Diode_SMD:D_SOD-123, B.Cu at (174.0, 12.1)
- added D2103: BAT48ZFILM, Diode_SMD:D_SOD-123, B.Cu at (174.0, 16.5)
- added D2104: BAT48ZFILM, Diode_SMD:D_SOD-123, B.Cu at (180.3, 16.5)
- added D301: 1N4148W, Diode_SMD:D_SOD-123, B.Cu at (85.1, 143.5)
- added D302: 1N4148W, Diode_SMD:D_SOD-123, B.Cu at (90.8, 143.5)
- added D501: D_Schottky, Diode_SMD:D_SOD-123, B.Cu at (166.9, 193.7)
- added D502: D_Schottky, Diode_SMD:D_SOD-123, B.Cu at (166.9, 189.2)
- added J101: ribbon_port, Connector_Molex:Molex_KK-254_AE-6410-03A_1x03_P2.54mm_Vertical, B.Cu at (195.6, 147.3)
- added J102: modosc_port, Connector_Molex:Molex_KK-254_AE-6410-02A_1x02_P2.54mm_Vertical, B.Cu at (195.6, 130.2)
- added J103: ADSR_port, Connector_Molex:Molex_KK-254_AE-6410-03A_1x03_P2.54mm_Vertical, B.Cu at (196.8, 17.1)
- added J104: S&H_port, Connector_Molex:Molex_KK-254_AE-6410-06A_1x06_P2.54mm_Vertical, B.Cu at (196.8, 59.1)
- added J105: ext_con, Connector_Molex:Molex_KK-254_AE-6410-03A_1x03_P2.54mm_Vertical, B.Cu at (67.3, -5.06)
- added J106: vcf_port, Connector_Molex:Molex_KK-254_AE-6410-03A_1x03_P2.54mm_Vertical, B.Cu at (196.8, 1.27)
- added J2301: power_entry, Connector_IDC:IDC-Header_2x05_P2.54mm_Vertical, B.Cu at (127.0, 186.6)
- added J501: aux_pwm, Connector_PinHeader_2.54mm:PinHeader_1x02_P2.54mm_Vertical, B.Cu at (157.5, 178.4)
- added Q1101: MMBT3904, Package_TO_SOT_SMD:SOT-23, B.Cu at (75.9, 92.1)
- added Q1102: MMBT3904, Package_TO_SOT_SMD:SOT-23, B.Cu at (70.5, 92.1)
- added Q1901: MMBT3904, Package_TO_SOT_SMD:SOT-23, B.Cu at (102.9, 15.2)
- added Q1902: MMBT3904, Package_TO_SOT_SMD:SOT-23, B.Cu at (108.6, 15.2)
- added Q401: 2N7002, Package_TO_SOT_SMD:SOT-23, B.Cu at (133.3, 146.7)
- added R1001: 15k, Resistor_SMD:R_0805_2012Metric, B.Cu at (49.5, 116.2)
- added R1002: 15k, Resistor_SMD:R_0805_2012Metric, B.Cu at (49.5, 112.4)
- added R1003: 7k5, Resistor_SMD:R_0805_2012Metric, B.Cu at (49.5, 108.6)
- added R1004: 120k, Resistor_SMD:R_0805_2012Metric, B.Cu at (49.5, 101.0)
- added R1005: 15k, Resistor_SMD:R_0805_2012Metric, B.Cu at (49.5, 104.8)
- added R1006: 120k, Resistor_SMD:R_0805_2012Metric, B.Cu at (55.2, 108.6)
- added R1101: 27k, Resistor_SMD:R_0805_2012Metric, B.Cu at (75.6, 101.0)
- added R1102: 2k2, Resistor_SMD:R_0805_2012Metric, B.Cu at (70.5, 101.0)
- added R1103: 10k, Resistor_SMD:R_0805_2012Metric, B.Cu at (75.6, 104.8)
- added R1104: 390, Resistor_SMD:R_0805_2012Metric, B.Cu at (75.6, 97.2)
- added R1105: 18k, Resistor_SMD:R_0805_2012Metric, B.Cu at (66.0, 86.4)
- added R1106: 10k, Resistor_SMD:R_0805_2012Metric, B.Cu at (75.6, 108.6)
- added R1107: 2k2, Resistor_SMD:R_0805_2012Metric, B.Cu at (70.5, 97.2)
- added R1108: 12k, Resistor_SMD:R_0805_2012Metric, B.Cu at (75.6, 112.4)
- added R1109: 12k, Resistor_SMD:R_0805_2012Metric, B.Cu at (70.5, 108.6)
- added R1201: 10k, Resistor_SMD:R_0805_2012Metric, B.Cu at (70.5, 112.4)
- added R1202: R, Resistor_SMD:R_0805_2012Metric, B.Cu at (75.6, 116.2)
- added R1203: R, Resistor_SMD:R_0805_2012Metric, B.Cu at (75.6, 120.0)
- added R1204: 10M, Resistor_SMD:R_0805_2012Metric, B.Cu at (70.5, 116.2)
- added R1205: 2k2, Resistor_SMD:R_0805_2012Metric, B.Cu at (70.5, 123.8)
- added R1301: 10k, Resistor_SMD:R_0805_2012Metric, B.Cu at (58.5, 149.5)
- added R1302: 10k, Resistor_SMD:R_0805_2012Metric, B.Cu at (58.5, 145.7)
- added R1401: 2M2, Resistor_SMD:R_0805_2012Metric, B.Cu at (76.1, 9.53)
- added R1501: 180k, Resistor_SMD:R_0805_2012Metric, B.Cu at (76.8, 72.4)
- added R1502: 200k, Resistor_SMD:R_0805_2012Metric, B.Cu at (76.8, 64.8)
- added R1503: 200k, Resistor_SMD:R_0805_2012Metric, B.Cu at (76.8, 68.6)
- added R1504: 100k, Resistor_SMD:R_0805_2012Metric, B.Cu at (76.8, 61.0)
- added R1505: 100k, Resistor_SMD:R_0805_2012Metric, B.Cu at (71.1, 61.0)
- added R1506: 100k, Resistor_SMD:R_0805_2012Metric, B.Cu at (71.1, 64.8)
- added R1601: 8k2, Resistor_SMD:R_0805_2012Metric, B.Cu at (81.3, 5.71)
- added R1602: 2k7, Resistor_SMD:R_0805_2012Metric, B.Cu at (81.3, 9.53)
- added R1603: 10k, Resistor_SMD:R_0805_2012Metric, B.Cu at (76.1, 5.71)
- added R1604: 120k, Resistor_SMD:R_0805_2012Metric, B.Cu at (76.1, 1.91)
- added R1605: 100k, Resistor_SMD:R_0805_2012Metric, B.Cu at (76.1, 13.3)
- added R1606: 1k, Resistor_SMD:R_0805_2012Metric, B.Cu at (76.2, 25.4)
- added R1607: 100k, Resistor_SMD:R_0805_2012Metric, B.Cu at (60.9, 9.53)
- added R1608: 100k, Resistor_SMD:R_0805_2012Metric, B.Cu at (61.0, 5.71)
- added R1609: 51k, Resistor_SMD:R_0805_2012Metric, B.Cu at (60.9, 24.8)
- added R1610: 1k, Resistor_SMD:R_0805_2012Metric, B.Cu at (61.0, 21.0)
- added R1611: 100k, Resistor_SMD:R_0805_2012Metric, B.Cu at (55.8, 5.71)
- added R1612: 180k, Resistor_SMD:R_0805_2012Metric, B.Cu at (55.8, 13.3)
- added R1613: 100k, Resistor_SMD:R_0805_2012Metric, B.Cu at (55.8, 17.1)
- added R1614: 200k, Resistor_SMD:R_0805_2012Metric, B.Cu at (55.8, 9.53)
- added R1615: 100k, Resistor_SMD:R_0805_2012Metric, B.Cu at (61.0, 13.3)
- added R1701: 33k, Resistor_SMD:R_0805_2012Metric, B.Cu at (76.8, 57.1)
- added R1702: 100k, Resistor_SMD:R_0805_2012Metric, B.Cu at (71.1, 57.1)
- added R1801: 15k, Resistor_SMD:R_0805_2012Metric, B.Cu at (49.5, 64.8)
- added R1802: 15k, Resistor_SMD:R_0805_2012Metric, B.Cu at (49.5, 61.0)
- added R1803: 7k5, Resistor_SMD:R_0805_2012Metric, B.Cu at (49.5, 57.1)
- added R1804: 120k, Resistor_SMD:R_0805_2012Metric, B.Cu at (49.5, 49.5)
- added R1805: 15k, Resistor_SMD:R_0805_2012Metric, B.Cu at (49.5, 53.3)
- added R1806: 120k, Resistor_SMD:R_0805_2012Metric, B.Cu at (54.6, 57.1)
- added R1901: 27k, Resistor_SMD:R_0805_2012Metric, B.Cu at (103.5, 20.3)
- added R1902: 2k2, Resistor_SMD:R_0805_2012Metric, B.Cu at (103.5, 24.1)
- added R1903: 10k, Resistor_SMD:R_0805_2012Metric, B.Cu at (108.6, 27.9)
- added R1904: 390, Resistor_SMD:R_0805_2012Metric, B.Cu at (108.6, 20.3)
- added R1905: 18k, Resistor_SMD:R_0805_2012Metric, B.Cu at (117.1, 27.9)
- added R1906: 10k, Resistor_SMD:R_0805_2012Metric, B.Cu at (108.6, 31.8)
- added R1907: 2k2, Resistor_SMD:R_0805_2012Metric, B.Cu at (108.6, 24.1)
- added R1908: 12k, Resistor_SMD:R_0805_2012Metric, B.Cu at (108.6, 35.6)
- added R1909: 12k, Resistor_SMD:R_0805_2012Metric, B.Cu at (103.5, 31.8)
- added R2001: 10k, Resistor_SMD:R_0805_2012Metric, B.Cu at (154.9, 36.2)
- added R2002: 100k, Resistor_SMD:R_0805_2012Metric, B.Cu at (154.9, 32.4)
- added R2003: 10M, Resistor_SMD:R_0805_2012Metric, B.Cu at (149.2, 36.2)
- added R2004: 100k, Resistor_SMD:R_0805_2012Metric, B.Cu at (149.2, 32.4)
- added R2005: 200k, Resistor_SMD:R_0805_2012Metric, B.Cu at (154.9, 21.0)
- added R2006: 200k, Resistor_SMD:R_0805_2012Metric, B.Cu at (154.9, 24.8)
- added R2007: 2k, Resistor_SMD:R_0805_2012Metric, B.Cu at (134.0, 31.1)
- added R2008: 100k, Resistor_SMD:R_0805_2012Metric, B.Cu at (149.2, 21.0)
- added R2009: 100k, Resistor_SMD:R_0805_2012Metric, B.Cu at (154.9, 17.1)
- added R201: 150k, Resistor_SMD:R_0805_2012Metric, B.Cu at (106.7, 128.3)
- added R2010: 100k, Resistor_SMD:R_0805_2012Metric, B.Cu at (149.2, 17.1)
- added R2011: 100k, Resistor_SMD:R_0805_2012Metric, B.Cu at (128.9, 24.8)
- added R2012: 100k, Resistor_SMD:R_0805_2012Metric, B.Cu at (128.9, 21.0)
- added R2013: 20k, Resistor_SMD:R_0805_2012Metric, B.Cu at (134.0, 21.0)
- added R2014: 220k, Resistor_SMD:R_0805_2012Metric, B.Cu at (128.9, 13.3)
- added R2015: 100k, Resistor_SMD:R_0805_2012Metric, B.Cu at (128.9, 17.1)
- added R2016: 180k, Resistor_SMD:R_0805_2012Metric, B.Cu at (134.0, 17.1)
- added R202: 56k, Resistor_SMD:R_0805_2012Metric, B.Cu at (116.8, 132.1)
- added R203: 120k, Resistor_SMD:R_0805_2012Metric, B.Cu at (111.8, 128.3)
- added R204: 100k, Resistor_SMD:R_0805_2012Metric, B.Cu at (167.0, 174.0)
- added R205: 100k, Resistor_SMD:R_0805_2012Metric, B.Cu at (167.0, 170.2)
- added R206: 200k, Resistor_SMD:R_0805_2012Metric, B.Cu at (167.0, 166.4)
- added R2101: 100k, Resistor_SMD:R_0805_2012Metric, B.Cu at (170.8, 60.2)
- added R2102: 100k, Resistor_SMD:R_0805_2012Metric, B.Cu at (170.8, 52.5)
- added R2103: 100k, Resistor_SMD:R_0805_2012Metric, B.Cu at (155.6, 60.2)
- added R2104: 330, Resistor_SMD:R_0805_2012Metric, B.Cu at (170.8, 44.9)
- added R2105: 100k, Resistor_SMD:R_0805_2012Metric, B.Cu at (155.6, 52.5)
- added R2106: 330, Resistor_SMD:R_0805_2012Metric, B.Cu at (155.6, 44.9)
- added R2107: 100k, Resistor_SMD:R_0805_2012Metric, B.Cu at (170.8, 56.4)
- added R2108: 100k, Resistor_SMD:R_0805_2012Metric, B.Cu at (83.2, 29.2)
- added R2109: 100k, Resistor_SMD:R_0805_2012Metric, B.Cu at (155.6, 56.4)
- added R2110: 100k, Resistor_SMD:R_0805_2012Metric, B.Cu at (88.3, 29.2)
- added R2111: R, Resistor_SMD:R_0805_2012Metric, B.Cu at (83.2, 25.4)
- added R2112: 100k, Resistor_SMD:R_0805_2012Metric, B.Cu at (88.3, 25.4)
- added R2201: 100k, Resistor_SMD:R_0805_2012Metric, B.Cu at (193.7, 93.3)
- added R2202: 100k, Resistor_SMD:R_0805_2012Metric, B.Cu at (188.6, 104.8)
- added R2203: 100k, Resistor_SMD:R_0805_2012Metric, B.Cu at (188.6, 101.0)
- added R2204: 100k, Resistor_SMD:R_0805_2012Metric, B.Cu at (193.7, 101.0)
- added R2205: 100k, Resistor_SMD:R_0805_2012Metric, B.Cu at (193.7, 104.8)
- added R2206: 100k, Resistor_SMD:R_0805_2012Metric, B.Cu at (193.7, 97.2)
- added R2207: 82k, Resistor_SMD:R_0805_2012Metric, B.Cu at (188.6, 97.2)
- added R2301: 1k8, Resistor_SMD:R_0805_2012Metric, B.Cu at (91.4, 118.7)
- added R2302: 4k7, Resistor_SMD:R_0805_2012Metric, B.Cu at (173.4, 104.8)
- added R2303: 10k, Resistor_SMD:R_0805_2012Metric, B.Cu at (173.4, 101.0)
- added R2304: 10k, Resistor_SMD:R_0805_2012Metric, B.Cu at (173.4, 97.2)
- added R301: 10k, Resistor_SMD:R_0805_2012Metric, B.Cu at (86.4, 139.7)
- added R302: 10k, Resistor_SMD:R_0805_2012Metric, B.Cu at (91.4, 139.7)
- added R303: 100K, Resistor_SMD:R_0805_2012Metric, B.Cu at (101.6, 128.3)
- added R304: 100K, Resistor_SMD:R_0805_2012Metric, B.Cu at (116.8, 143.5)
- added R305: 1m, Resistor_SMD:R_0805_2012Metric, B.Cu at (121.9, 135.9)
- added R306: 100K, Resistor_SMD:R_0805_2012Metric, B.Cu at (121.9, 132.1)
- added R307: 100K, Resistor_SMD:R_0805_2012Metric, B.Cu at (121.9, 143.5)
- added R308: 100K, Resistor_SMD:R_0805_2012Metric, B.Cu at (121.9, 139.7)
- added R309: 100K, Resistor_SMD:R_0805_2012Metric, B.Cu at (116.8, 128.3)
- added R310: 100K, Resistor_SMD:R_0805_2012Metric, B.Cu at (121.9, 128.3)
- added R311: 100k, Resistor_SMD:R_0805_2012Metric, B.Cu at (116.8, 139.7)
- added R312: 270K, Resistor_SMD:R_0805_2012Metric, B.Cu at (116.8, 135.9)
- added R313: 47K, Resistor_SMD:R_0805_2012Metric, B.Cu at (91.4, 132.1)
- added R314: 270, Resistor_SMD:R_0805_2012Metric, B.Cu at (86.4, 128.3)
- added R315: 470K, Resistor_SMD:R_0805_2012Metric, B.Cu at (91.4, 135.9)
- added R316: 4k7, Resistor_SMD:R_0805_2012Metric, B.Cu at (96.5, 128.3)
- added R317: 100k, Resistor_SMD:R_0805_2012Metric, B.Cu at (95.2, 0.00)
- added R318: 3K9, Resistor_SMD:R_0805_2012Metric, B.Cu at (111.8, 132.1)
- added R319: 4K7, Resistor_SMD:R_0805_2012Metric, B.Cu at (111.8, 135.9)
- added R320: 12K, Resistor_SMD:R_0805_2012Metric, B.Cu at (111.8, 143.5)
- added R321: 4K7, Resistor_SMD:R_0805_2012Metric, B.Cu at (111.8, 139.7)
- added R322: 10k, Resistor_SMD:R_0805_2012Metric, B.Cu at (91.4, 128.3)
- added R401: 100k, Resistor_SMD:R_0805_2012Metric, B.Cu at (132.7, 134.0)
- added R402: 100k, Resistor_SMD:R_0805_2012Metric, B.Cu at (132.7, 130.2)
- added R403: 100k, Resistor_SMD:R_0805_2012Metric, B.Cu at (138.4, 134.0)
- added R404: 100, Resistor_SMD:R_0805_2012Metric, B.Cu at (153.7, 149.2)
- added R405: 100k, Resistor_SMD:R_0805_2012Metric, B.Cu at (138.4, 149.2)
- added R406: 10k, Resistor_SMD:R_0805_2012Metric, B.Cu at (138.4, 145.4)
- added R407: 20k, Resistor_SMD:R_0805_2012Metric, B.Cu at (132.7, 141.6)
- added R408: 20k, Resistor_SMD:R_0805_2012Metric, B.Cu at (132.7, 137.8)
- added R409: 20k, Resistor_SMD:R_0805_2012Metric, B.Cu at (138.4, 137.8)
- added R501: 100k, Resistor_SMD:R_0805_2012Metric, B.Cu at (182.2, 170.2)
- added R502: 270k, Resistor_SMD:R_0805_2012Metric, B.Cu at (182.2, 166.4)
- added R503: 100, Resistor_SMD:R_0805_2012Metric, B.Cu at (182.8, 183.7)
- added R504: 10k, Resistor_SMD:R_0805_2012Metric, B.Cu at (182.8, 186.7)
- added R505: 100k, Resistor_SMD:R_0805_2012Metric, B.Cu at (182.2, 174.0)
- added R506: 220k, Resistor_SMD:R_0805_2012Metric, B.Cu at (161.6, 185.4)
- added R507: 180k, Resistor_SMD:R_0805_2012Metric, B.Cu at (161.6, 181.6)
- added R508: 180k, Resistor_SMD:R_0805_2012Metric, B.Cu at (161.6, 177.8)
- added R509: 100k, Resistor_SMD:R_0805_2012Metric, B.Cu at (166.9, 177.8)
- added R510: 1k, Resistor_SMD:R_0805_2012Metric, B.Cu at (166.9, 185.4)
- added R601: 1M5, Resistor_SMD:R_0805_2012Metric, B.Cu at (131.0, 68.6)
- added R701: 180k, Resistor_SMD:R_0805_2012Metric, B.Cu at (159.4, 145.4)
- added R702: 200k, Resistor_SMD:R_0805_2012Metric, B.Cu at (159.4, 137.8)
- added R703: 200k, Resistor_SMD:R_0805_2012Metric, B.Cu at (159.4, 141.6)
- added R704: 100k, Resistor_SMD:R_0805_2012Metric, B.Cu at (159.4, 134.0)
- added R705: 100k, Resistor_SMD:R_0805_2012Metric, B.Cu at (153.7, 137.8)
- added R706: 100k, Resistor_SMD:R_0805_2012Metric, B.Cu at (153.7, 141.6)
- added R801: 8k2, Resistor_SMD:R_0805_2012Metric, B.Cu at (136.0, 64.8)
- added R802: 2k7, Resistor_SMD:R_0805_2012Metric, B.Cu at (136.0, 68.6)
- added R803: 10k, Resistor_SMD:R_0805_2012Metric, B.Cu at (131.0, 64.8)
- added R804: 120k, Resistor_SMD:R_0805_2012Metric, B.Cu at (131.0, 61.0)
- added R805: 100k, Resistor_SMD:R_0805_2012Metric, B.Cu at (131.0, 72.4)
- added R806: 1k, Resistor_SMD:R_0805_2012Metric, B.Cu at (131.0, 84.5)
- added R807: 100k, Resistor_SMD:R_0805_2012Metric, B.Cu at (115.6, 68.6)
- added R808: 100k, Resistor_SMD:R_0805_2012Metric, B.Cu at (115.7, 64.8)
- added R809: 51k, Resistor_SMD:R_0805_2012Metric, B.Cu at (115.7, 83.8)
- added R810: 1k, Resistor_SMD:R_0805_2012Metric, B.Cu at (115.7, 80.0)
- added R811: 100k, Resistor_SMD:R_0805_2012Metric, B.Cu at (110.6, 64.8)
- added R812: 180k, Resistor_SMD:R_0805_2012Metric, B.Cu at (110.6, 72.4)
- added R813: 100k, Resistor_SMD:R_0805_2012Metric, B.Cu at (110.6, 76.2)
- added R814: 200k, Resistor_SMD:R_0805_2012Metric, B.Cu at (110.6, 68.6)
- added R815: 100k, Resistor_SMD:R_0805_2012Metric, B.Cu at (115.7, 72.4)
- added R901: 33k, Resistor_SMD:R_0805_2012Metric, B.Cu at (159.4, 130.2)
- added R902: 100k, Resistor_SMD:R_0805_2012Metric, B.Cu at (153.7, 134.0)
- added RV1101: 50k, Potentiometer_THT:Potentiometer_Bourns_3296W_Vertical, B.Cu at (71.1, 79.2)
- added RV1102: 50k, Potentiometer_THT:Potentiometer_Bourns_3296W_Vertical, B.Cu at (71.1, 85.7)
- added RV1501: 50k, Potentiometer_THT:Potentiometer_Bourns_3296W_Vertical, B.Cu at (83.2, 67.9)
- added RV1601: 50k, Potentiometer_THT:Potentiometer_Bourns_3296W_Vertical, B.Cu at (45.1, 16.5)
- added RV1602: 5k, Potentiometer_THT:Potentiometer_Bourns_3296W_Vertical, B.Cu at (45.1, 8.89)
- added RV1901: 50k, Potentiometer_THT:Potentiometer_Bourns_3296W_Vertical, B.Cu at (115.6, 15.9)
- added RV1902: 50k, Potentiometer_THT:Potentiometer_Bourns_3296W_Vertical, B.Cu at (115.6, 22.3)
- added RV2001: 50k, Potentiometer_THT:Potentiometer_Bourns_3296W_Vertical, B.Cu at (128.3, 38.1)
- added RV201: 10k, Potentiometer_THT:Potentiometer_Alpha_RD901F-40-00D_Single_Vertical, F.Cu at (48.3, 83.8)
- added RV202: 10k, Potentiometer_THT:Potentiometer_Alpha_RD901F-40-00D_Single_Vertical, F.Cu at (48.3, 33.0)
- added RV203: 100k, Potentiometer_THT:Potentiometer_Alpha_RD901F-40-00D_Single_Vertical, F.Cu at (92.8, 172.7)
- added RV204: 100k, Potentiometer_THT:Potentiometer_Alpha_RD901F-40-00D_Single_Vertical, F.Cu at (42.0, 172.7)
- added RV205: 100k, Potentiometer_THT:Potentiometer_Alpha_RD901F-40-00D_Single_Vertical, F.Cu at (67.3, 147.3)
- added RV2101: 20k, Potentiometer_THT:Potentiometer_Bourns_3296W_Vertical, B.Cu at (177.2, 56.4)
- added RV2102: 20k, Potentiometer_THT:Potentiometer_Bourns_3296W_Vertical, B.Cu at (177.2, 48.1)
- added RV2201: 100k, Potentiometer_THT:Potentiometer_Alpha_RD901F-40-00D_Single_Vertical, F.Cu at (143.6, 7.63)
- added RV2202: 100k, Potentiometer_THT:Potentiometer_Alpha_RD901F-40-00D_Single_Vertical, F.Cu at (143.6, 58.4)
- added RV2203: 100k, Potentiometer_THT:Potentiometer_Alpha_RD901F-40-00D_Single_Vertical, F.Cu at (143.6, 109.2)
- added RV2204: 100k, Potentiometer_THT:Potentiometer_Alpha_RD901F-40-00D_Single_Vertical, F.Cu at (188.0, 33.0)
- added RV2205: 100k, Potentiometer_THT:Potentiometer_Alpha_RD901F-40-00D_Single_Vertical, F.Cu at (188.0, 83.8)
- added RV301: 5k, Potentiometer_THT:Potentiometer_Bourns_3296W_Vertical, B.Cu at (99.0, 149.9)
- added RV302: 5k, Potentiometer_THT:Potentiometer_Bourns_3296W_Vertical, B.Cu at (88.9, 149.9)
- added RV303: 5k, Potentiometer_THT:Potentiometer_Bourns_3296W_Vertical, B.Cu at (109.2, 149.9)
- added RV501: 100k, Potentiometer_THT:Potentiometer_Alpha_RD901F-40-00D_Single_Vertical, F.Cu at (143.6, 172.7)
- added RV502: 100k, Potentiometer_THT:Potentiometer_Alpha_RD901F-40-00D_Single_Vertical, F.Cu at (194.3, 172.7)
- added RV503: 100k, Potentiometer_THT:Potentiometer_Alpha_RD901F-40-00D_Single_Vertical, F.Cu at (168.9, 147.3)
- added RV701: 50k, Potentiometer_THT:Potentiometer_Bourns_3296W_Vertical, B.Cu at (159.4, 151.1)
- added RV801: 50k, Potentiometer_THT:Potentiometer_Bourns_3296W_Vertical, B.Cu at (99.8, 76.2)
- added RV802: 5k, Potentiometer_THT:Potentiometer_Bourns_3296W_Vertical, B.Cu at (99.8, 68.6)
- added SW1401: SW_SPDT_CO, custom_footprints:SPDT_mini_toggle, F.Cu at (120.7, 101.6)
- added SW1402: SR1712F-0204, custom_footprints:SR1712F_rotary_switch, F.Cu at (95.2, 101.6)
- added SW201: SW_SPDT_CO, custom_footprints:SPDT_mini_toggle, F.Cu at (44.5, 190.5)
- added SW202: SW_SPDT_CO, custom_footprints:SPDT_mini_toggle, F.Cu at (69.8, 190.5)
- added SW203: SW_SPDT_CO, custom_footprints:SPDT_mini_toggle, F.Cu at (95.2, 190.5)
- added SW2101: SW_DPDT_CO, custom_footprints:DPDT_mini_toggle, F.Cu at (165.1, 25.4)
- added SW2201: SW_SPDT, custom_footprints:SPDT_mini_toggle, F.Cu at (120.7, 0.00)
- added SW2202: SW_SPDT, custom_footprints:SPDT_mini_toggle, F.Cu at (165.1, 76.2)
- added SW301: SR1712F-0204, custom_footprints:SR1712F_rotary_switch, F.Cu at (95.2, 0.00)
- added SW601: SW_DPDT_CO, custom_footprints:DPDT_mini_toggle, F.Cu at (120.7, 50.8)
- added SW602: SR1712F-0204, custom_footprints:SR1712F_rotary_switch, F.Cu at (95.2, 50.8)
- added TP101: pwm_cv, TestPoint:TestPoint_Keystone_5000-5004_Miniature, B.Cu at (71.1, 172.7)
- added TP102: oct_0, TestPoint:TestPoint_Keystone_5000-5004_Miniature, B.Cu at (84.4, 177.8)
- added TP103: oct_1, TestPoint:TestPoint_Keystone_5000-5004_Miniature, B.Cu at (71.3, 177.8)
- added TP104: oct_2, TestPoint:TestPoint_Keystone_5000-5004_Miniature, B.Cu at (80.0, 177.8)
- added TP105: ring_mod, TestPoint:TestPoint_Keystone_5000-5004_Miniature, B.Cu at (75.7, 177.8)
- added TP2301: V+, TestPoint:TestPoint_Keystone_5000-5004_Miniature, B.Cu at (76.8, 172.7)
- added TP2302: V-, TestPoint:TestPoint_Keystone_5000-5004_Miniature, B.Cu at (83.8, 172.7)
- added TP2303: GND, TestPoint:TestPoint_Bridge_Pitch7.62mm_Drill1.3mm, B.Cu at (85.1, 184.7)
- added TR2101: Triad_TY_141P, custom_footprints:Triad_TY-141P, B.Cu at (177.2, 26.7)
- added TR2102: Triad_TY_141P, custom_footprints:Triad_TY-141P, B.Cu at (177.2, 1.91)
- added U1: TL074, Package_SO:SOIC-14_3.9x8.7mm_P1.27mm, B.Cu at (174.6, 174.0)
- added U10: DG413xY, Package_SO:SOIC-16_3.9x9.9mm_P1.27mm, B.Cu at (50.8, 132.1)
- added U11: TL074, Package_SO:SOIC-14_3.9x8.7mm_P1.27mm, B.Cu at (62.9, 61.0)
- added U12: TL074, Package_SO:SOIC-14_3.9x8.7mm_P1.27mm, B.Cu at (68.6, 10.8)
- added U13: LM311, Package_SO:SOIC-8_3.9x4.9mm_P1.27mm, B.Cu at (68.6, 23.5)
- added U14: TL074, Package_SO:SOIC-14_3.9x8.7mm_P1.27mm, B.Cu at (95.9, 27.9)
- added U15: TL074, Package_SO:SOIC-14_3.9x8.7mm_P1.27mm, B.Cu at (141.6, 34.3)
- added U16: TL074, Package_SO:SOIC-14_3.9x8.7mm_P1.27mm, B.Cu at (141.6, 17.1)
- added U17: NE5532, Package_SO:SOIC-8_3.9x4.9mm_P1.27mm, B.Cu at (163.2, 50.8)
- added U18: TL072, Package_SO:SOIC-8_3.9x4.9mm_P1.27mm, B.Cu at (181.0, 98.4)
- added U2: TL074, Package_SO:SOIC-14_3.9x8.7mm_P1.27mm, B.Cu at (146.1, 134.0)
- added U2301: L78L05_SOT89, Package_TO_SOT_SMD:SOT-89-3, B.Cu at (109.2, 175.9)
- added U2302: L79L05_SOT89, Package_TO_SOT_SMD:SOT-89-3, B.Cu at (109.2, 186.7)
- added U2303: LM4040C-2.5, Package_TO_SOT_SMD:SOT-23, B.Cu at (86.4, 120.7)
- added U2304: LM4040DBZ-5, Package_TO_SOT_SMD:SOT-23, B.Cu at (168.3, 107.3)
- added U3: LM311, Package_SO:SOIC-8_3.9x4.9mm_P1.27mm, B.Cu at (146.1, 149.2)
- added U4: SSI2130, custom_footprints:PQN32_HandSoldering, B.Cu at (101.6, 137.2)
- added U5: 4013, Package_SO:SOIC-14_3.9x8.7mm_P1.27mm, B.Cu at (62.9, 45.1)
- added U6: TL074, Package_SO:SOIC-14_3.9x8.7mm_P1.27mm, B.Cu at (123.3, 69.8)
- added U7: LM311, Package_SO:SOIC-8_3.9x4.9mm_P1.27mm, B.Cu at (123.3, 82.5)
- added U8: TL074, Package_SO:SOIC-14_3.9x8.7mm_P1.27mm, B.Cu at (62.9, 111.8)
- added U9: LM555xM, Package_SO:SOIC-8_3.9x4.9mm_P1.27mm, B.Cu at (50.8, 146.7)
Routing:
- net Net-(C802-Pad2): track 0.00 -> 47.4 mm
- net Net-(C1602-Pad2): track 0.00 -> 47.4 mm
- net Net-(C502-Pad1): track 0.00 -> 22.6 mm
- net Net-(C801-Pad1): track 0.00 -> 21.5 mm
- net Net-(C1601-Pad1): track 0.00 -> 21.5 mm
- net Net-(R811-Pad2): track 0.00 -> 21.4 mm
- net Net-(R1611-Pad2): track 0.00 -> 21.4 mm
- net /sub_osc_1/saw_animator_1/RATE_R_1: track 0.00 -> 20.7 mm
- net /sub_osc_2/saw_animator_2/RATE_R_1: track 0.00 -> 20.3 mm
- net /PWM_LFO_TRI: track 0.00 -> 20.0 mm
- net Net-(C502-Pad2): track 0.00 -> 19.1 mm
- net Net-(C201-Pad2): track 0.00 -> 18.2 mm
- net Net-(C201-Pad1): track 0.00 -> 15.7 mm
- net Net-(R1608-Pad2): track 0.00 -> 14.1 mm
- net Net-(R808-Pad2): track 0.00 -> 14.1 mm
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Other:
- board text removed: "Crosshairs show the locations of the pots and switches. Double check before layout and ordering!"
