File: summer_2022_refurb/main_VCO_board/kicad_6_docs/main_VCO.kicad_sch (KiCad schematic)
At the start: 11 parts

Commit message: Main VCO progress
Parts:
- added C?: C, symbol Device:C
- added C?: 220n, symbol Device:C
- added R? (x2): 100k, symbol Device:R
- added R?: 200k, symbol Device:R
- added U?: TL072, symbol Amplifier_Operational:TL072
- SW? (x3): value SW_SPDT_MSM -> SW_SPDT_CO
Connections:
- net GND: now also U?.3 (+)
- net OUT: now also C?.2
- net VCO_core/SWITCHED_OUT: now also R?.1, R?.1
- new net: C?.1, R?.1, R?.2, R?.2, U?.2 (-)
- new net: C?.1, C?.2, R?.2, U?.1
Other:
- removed sheet level_shifter_1
- note added: "[-1.25, +1.25v] in"
- note added: "[-5v, +5v] out"
- note added: "[0, +2.5v]"
- note added: "[0, +5v]"
- title: (none) -> Josh Ox Ribon Synth Main VCO board

Commit message: Progress on main VCO, schem getting close but not done
Parts:
- removed U?: TL072, symbol Amplifier_Operational:TL072
- added U1: TL074, symbol Amplifier_Operational:TL074
- gave numbers to parts that had none: 16
Connections:
- net GND: now also U1.12 (+)
- net at C201.1, R204.2, R205.2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: now also U1.13 (-)
- net at C201.2, C202.1, R206.2: now also U1.14

Commit message: Main VCO rough parts placement
Parts:
- C201: footprint (none) -> Capacitor_SMD:C_0805_2012Metric
- C202: footprint (none) -> Capacitor_THT:C_Rect_L7.0mm_W2.5mm_P5.00mm
- R201, R202, R203, R204, R205, R206: footprint (none) -> Resistor_SMD:R_0805_2012Metric
- RV201, RV202, RV203, RV204, RV205: footprint (none) -> Potentiometer_THT:Potentiometer_Alpha_RD901F-40-00D_Single_Vertical
- SW201, SW202, SW203: footprint (none) -> custom_footprints:SPDT_mini_toggle
- U1: footprint (none) -> Package_SO:SOIC-14_3.9x8.7mm_P1.27mm
Changed lines of the file:
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@@
     (property "Reference" "SW201" (id 0) (at 58.293 76.2 0))
     (property "Value" "SW_SPDT_CO" (id 1) (at 58.293 78.74 0))
-    (property "Footprint" "" (id 2) (at 58.42 83.82 0)
+    (property "Footprint" "custom_footprints:SPDT_mini_toggle" (id 2) (at 58.42 83.82 0)
       (effects (font (size 1.27 1.27)) hide)
     )
@@
     (property "Reference" "C201" (id 0) (at 220.98 22.86 90))
     (property "Value" "C" (id 1) (at 220.98 25.4 90))
-    (property "Footprint" "" (id 2) (at 224.79 29.5148 0)
+    (property "Footprint" "Capacitor_SMD:C_0805_2012Metric" (id 2) (at 224.79 29.5148 0)
       (effects (font (size 1.27 1.27)) hide)
     )
@@
     (property "Reference" "R204" (id 0) (at 199.39 40.64 90))
     (property "Value" "100k" (id 1) (at 199.39 43.18 90))
-    (property "Footprint" "" (id 2) (at 199.39 48.768 90)
+    (property "Footprint" "Resistor_SMD:R_0805_2012Metric" (id 2) (at 199.39 48.768 90)
       (effects (font (size 1.27 1.27)) hide)
     )
@@
       (effects (font (size 1.27 1.27)) (justify left))
     )
-    (property "Footprint" "" (id 2) (at 62.992 166.37 90)
+    (property "Footprint" "Resistor_SMD:R_0805_2012Metric" (id 2) (at 62.992 166.37 90)
       (effects (font (size 1.27 1.27)) hide)
     )
@@
       (effects (font (size 1.27 1.27)) (justify right))
     )
-    (property "Footprint" "" (id 2) (at 58.42 135.89 0)
+    (property "Footprint" "Potentiometer_THT:Potentiometer_Alpha_RD901F-40-00D_Single_Vertical" (id 2) (at 58.42 135.89 0)
       (effects (font (size 1.27 1.27)) hide)
     )
@@
     (property "Reference" "C202" (id 0) (at 237.49 44.45 90))
     (property "Value" "220n" (id 1) (at 237.49 46.99 90))
-    (property "Footprint" "" (id 2) (at 241.3 51.1048 0)
+    (property "Footprint" "Capacitor_THT:C_Rect_L7.0mm_W2.5mm_P5.00mm" (id 2) (at 241.3 51.1048 0)
       (effects (font (size 1.27 1.27)) hide)
     )
@@
       (effects (font (size 1.27 1.27)) (justify right))
     )
-    (property "Footprint" "" (id 2) (at 46.99 31.75 0)
+    (property "Footprint" "Potentiometer_THT:Potentiometer_Alpha_RD901F-40-00D_Single_Vertical" (id 2) (at 46.99 31.75 0)
       (effects (font (size 1.27 1.27)) hide)
     )
@@
     (property "Reference" "SW203" (id 0) (at 71.247 128.27 0))
     (property "Value" "SW_SPDT_CO" (id 1) (at 71.247 130.81 0))
-    (property "Footprint" "" (id 2) (at 71.12 135.89 0)
+    (property "Footprint" "custom_footprints:SPDT_mini_toggle" (id 2) (at 71.12 135.89 0)
       (effects (font (size 1.27 1.27)) hide)
     )
@@
       (effects (font (size 1.27 1.27)) (justify right))
     )
-    (property "Footprint" "" (id 2) (at 77.47 90.17 0)
+    (property "Footprint" "Potentiometer_THT:Potentiometer_Alpha_RD901F-40-00D_Single_Vertical" (id 2) (at 77.47 90.17 0)
       (effects (font (size 1.27 1.27)) hide)
     )
@@
       (effects (font (size 1.27 1.27)) (justify right))
     )
-    (property "Footprint" "" (id 2) (at 45.72 50.8 0)
+    (property "Footprint" "Potentiometer_THT:Potentiometer_Alpha_RD901F-40-00D_Single_Vertical" (id 2) (at 45.72 50.8 0)
       (effects (font (size 1.27 1.27)) hide)
     )
@@
     (property "Reference" "R206" (id 0) (at 220.98 35.56 90))
     (property "Value" "200k" (id 1) (at 220.98 38.1 90))
-    (property "Footprint" "" (id 2) (at 220.98 43.688 90)
+    (property "Footprint" "Resistor_SMD:R_0805_2012Metric" (id 2) (at 220.98 43.688 90)
       (effects (font (size 1.27 1.27)) hide)
     )
@@
     (property "Reference" "U1" (id 0) (at 223.52 60.96 0))
     (property "Value" "TL074" (id 1) (at 224.79 63.5 0))
-    (property "Footprint" "" (id 2) (at 219.71 57.15 0)
+    (property "Footprint" "Package_SO:SOIC-14_3.9x8.7mm_P1.27mm" (id 2) (at 219.71 57.15 0)
       (effects (font (size 1.27 1.27)) hide)
     )
@@
     (property "Reference" "SW202" (id 0) (at 58.293 97.79 0))
     (property "Value" "SW_SPDT_CO" (id 1) (at 58.293 100.33 0))
-    (property "Footprint" "" (id 2) (at 58.42 105.41 0)
+    (property "Footprint" "custom_footprints:SPDT_mini_toggle" (id 2) (at 58.42 105.41 0)
       (effects (font (size 1.27 1.27)) hide)
     )
@@
     (property "Reference" "R205" (id 0) (at 199.39 50.8 90))
     (property "Value" "100k" (id 1) (at 199.39 53.34 90))
-    (property "Footprint" "" (id 2) (at 199.39 58.928 90)
+    (property "Footprint" "Resistor_SMD:R_0805_2012Metric" (id 2) (at 199.39 58.928 90)
       (effects (font (size 1.27 1.27)) hide)
     )
@@
     (property "Reference" "R201" (id 0) (at 55.88 166.37 90))
     (property "Value" "150k" (id 1) (at 55.88 168.91 90))
-    (property "Footprint" "" (id 2) (at 55.88 174.498 90)
+    (property "Footprint" "Resistor_SMD:R_0805_2012Metric" (id 2) (at 55.88 174.498 90)
       (effects (font (size 1.27 1.27)) hide)
     )
@@
       (effects (font (size 1.27 1.27)) (justify left))
     )
-    (property "Footprint" "" (id 2) (at 60.452 179.07 90)
+    (property "Footprint" "Resistor_SMD:R_0805_2012Metric" (id 2) (at 60.452 179.07 90)
       (effects (font (size 1.27 1.27)) hide)
     )
@@
       (effects (font (size 1.27 1.27)) (justify right))
     )
-    (property "Footprint" "" (id 2) (at 77.47 111.76 0)
-      (effects (font (size 1.27 1.27)) hide)
-    )
+    (property "Footprint" "Potentiometer_THT:Potentiometer_Alpha_RD901F-40-00D_Single_Vertical" (id 2) (at 77.47 111.76 0)
+      (effects (font (size 1.27 1.27)) hide)
+    )

Commit message: Begin VCO pcb layout
Parts:
- renumbered U1 to U2
Connections:
- net GND: now also U2.3 (+); no longer U2.12 (+)
- net at C201.1, R204.2, R205.2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: now also U2.2 (-); no longer U2.13 (-)
- net at C201.2, C202.1, R206.2: now also U2.1; no longer U2.14
Changed lines of the file:
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@@
     (pin "2")
   )
-  (symbol (lib_id "Amplifier_Operational:TL074") (at 220.98 54.61 0) (mirror x) (unit 4)
+  (symbol (lib_id "Amplifier_Operational:TL074") (at 220.98 54.61 0) (mirror x) (unit 1)
     (in_bom yes) (on_board yes)
-    (property "Reference" "U1" (id 0) (at 223.52 60.96 0))
+    (property "Reference" "U2" (id 0) (at 223.52 60.96 0))
     (property "Value" "TL074" (id 1) (at 224.79 63.5 0))
     (property "Footprint" "Package_SO:SOIC-14_3.9x8.7mm_P1.27mm" (id 2) (at 219.71 57.15 0)
