File: summer_2022_refurb/ribbon_board/kicad_6_docs/ribbon_board.kicad_pcb (KiCad board)
At the start: 2 copper layers, 179 parts, among them J1 VCO_port, J2 VCF_port, J3 mod_osc_port, J301 ribbon, J4 ADSR_port, J5 S&H_port, J6 ext_port, J7 power_entry, SW1201 SW_SPDT, SW1301 SW_SPDT_MSM, SW1401 SW_SPDT_MSM, SW1501 SW_SPDT_MSM, SW1601 SW_SPDT_MSM, SW1701 SW_SPDT, SW201 SW_SPDT, U1 TL072, U10 TL072, U1002 TLC555xD, U1003 LF398_SOIC14, U1004 LF398_SOIC14, U2 TL072, U3 TL072, U301 L78L10_SOT89, U4 4081, U401 LF398_SOIC14, U5 4013, U6 40106, U601 LM358, U7 40106, U702 4017, U8 4081, U802 TLC555xD, U803 LF398_SOIC14, U804 LF398_SOIC14, U9 TL072

Commit message: Initial ribbon board layout
Parts:
- added REF**: OSHW-Logo_5.7x6mm_SilkScreen, Symbol:OSHW-Logo_5.7x6mm_SilkScreen, B.Cu at (52.5, 111.0)
- added kibuzzard-62AC7A9F: G***, kibuzzard-62AC7A9F, B.Cu at (51.3, 105.2)
- added kibuzzard-62B1F2D1: G***, kibuzzard-62B1F2D1, B.Cu at (158.8, 99.4)
- added kibuzzard-62B1F2D1: G***, kibuzzard-62B1F2D1, B.Cu at (181.6, 47.2)
- added kibuzzard-62B1F2D1: G***, kibuzzard-62B1F2D1, B.Cu at (26.9, 69.8)
- added kibuzzard-62B1F2D1: G***, kibuzzard-62B1F2D1, B.Cu at (27.0, 50.4)
- added kibuzzard-62B1F2D1: G***, kibuzzard-62B1F2D1, B.Cu at (81.3, 101.3)
- added kibuzzard-62B1F2D1: G***, kibuzzard-62B1F2D1, B.Cu at (27.0, 87.4)
- added kibuzzard-62B1F2D1: G***, kibuzzard-62B1F2D1, B.Cu at (166.6, 76.5)
- added kibuzzard-62B1F2D1: G***, kibuzzard-62B1F2D1, B.Cu at (106.7, 47.0)
- added kibuzzard-62B1F3ED: G***, kibuzzard-62B1F3ED, B.Cu at (28.0, 47.9)
- added kibuzzard-62B1F45D: G***, kibuzzard-62B1F45D, B.Cu at (27.3, 84.8)
- added kibuzzard-62B1F49A: G***, kibuzzard-62B1F49A, B.Cu at (29.6, 79.8)
- added kibuzzard-62B1F4B1: G***, kibuzzard-62B1F4B1, B.Cu at (29.6, 82.3)
- added kibuzzard-62B1F4C1: G***, kibuzzard-62B1F4C1, B.Cu at (29.0, 64.8)
- added kibuzzard-62B1F525: G***, kibuzzard-62B1F525, B.Cu at (83.8, 99.1)
- added kibuzzard-62B1F53B: G***, kibuzzard-62B1F53B, B.Cu at (86.4, 98.0)
- added kibuzzard-62B1F567: G***, kibuzzard-62B1F567, B.Cu at (29.5, 67.3)
- added kibuzzard-62B1F712: G***, kibuzzard-62B1F712, B.Cu at (186.7, 48.0)
- added kibuzzard-62B1F72D: G***, kibuzzard-62B1F72D, B.Cu at (109.2, 48.0)
- added kibuzzard-62B1F743: G***, kibuzzard-62B1F743, B.Cu at (111.8, 49.8)
- added kibuzzard-62B1F752: G***, kibuzzard-62B1F752, B.Cu at (114.3, 49.8)
- added kibuzzard-62B1F77F: G***, kibuzzard-62B1F77F, B.Cu at (116.8, 49.8)
- added kibuzzard-62B1F7DB: G***, kibuzzard-62B1F7DB, B.Cu at (189.2, 49.5)
- added kibuzzard-62B1F7F1: G***, kibuzzard-62B1F7F1, B.Cu at (184.2, 48.8)
- added kibuzzard-62B1F821: G***, kibuzzard-62B1F821, B.Cu at (185.4, 35.3)
- added kibuzzard-62B1F8A8: G***, kibuzzard-62B1F8A8, B.Cu at (111.8, 35.3)
- added kibuzzard-62B1F8CB: G***, kibuzzard-62B1F8CB, B.Cu at (15.0, 49.0)
- added kibuzzard-62B1F8F4: G***, kibuzzard-62B1F8F4, B.Cu at (15.0, 67.3)
- added kibuzzard-62B1F904: G***, kibuzzard-62B1F904, B.Cu at (15.0, 83.6)
- added kibuzzard-62B1F917: G***, kibuzzard-62B1F917, B.Cu at (83.8, 113.0)
- added kibuzzard-62B1F959: G***, kibuzzard-62B1F959, B.Cu at (163.8, 99.4)
- added kibuzzard-62B1F959: G***, kibuzzard-62B1F959, B.Cu at (162.3, 89.4)
- added kibuzzard-62B1F963: G***, kibuzzard-62B1F963, B.Cu at (168.7, 83.8)
- added kibuzzard-62B1F963: G***, kibuzzard-62B1F963, B.Cu at (153.7, 99.4)
- added kibuzzard-62B1F9D0: G***, kibuzzard-62B1F9D0, B.Cu at (158.8, 113.0)
- added kibuzzard-62B1FC16: G***, kibuzzard-62B1FC16, B.Cu at (51.8, 49.5)
- added kibuzzard-62B1FC43: G***, kibuzzard-62B1FC43, B.Cu at (51.6, 70.6)
- added kibuzzard-62B1FC58: G***, kibuzzard-62B1FC58, B.Cu at (51.6, 81.8)
- added kibuzzard-62B1FC81: G***, kibuzzard-62B1FC81, B.Cu at (23.1, 106.2)
- added kibuzzard-62B1FCCC: G***, kibuzzard-62B1FCCC, B.Cu at (101.1, 53.8)
- added kibuzzard-62B1FD45: G***, kibuzzard-62B1FD45, B.Cu at (200.7, 50.3)
- added kibuzzard-62B1FD51: G***, kibuzzard-62B1FD51, B.Cu at (201.2, 40.9)
- added kibuzzard-62B1FD62: G***, kibuzzard-62B1FD62, B.Cu at (93.7, 41.4)
- added kibuzzard-62B1FDDB: G***, kibuzzard-62B1FDDB, B.Cu at (171.4, 39.1)
- added kibuzzard-62B1FE6D: G***, kibuzzard-62B1FE6D, B.Cu at (199.4, 84.3)
- added kibuzzard-62B1FEB0: G***, kibuzzard-62B1FEB0, B.Cu at (23.1, 96.3)
- added kibuzzard-62B1FECC: G***, kibuzzard-62B1FECC, B.Cu at (137.2, 60.5)
- added kibuzzard-62B235EB: G***, kibuzzard-62B235EB, B.Cu at (107.3, 113.0)
- added kibuzzard-62B23681: G***, kibuzzard-62B23681, B.Cu at (198.6, 109.1)
- added kibuzzard-62B239A3: G***, kibuzzard-62B239A3, B.Cu at (61.3, 110.9)
- moved C5 380.5 mm to (64.0, 70.5)
- moved C6 380.5 mm to (64.0, 55.9)
- moved C7 380.5 mm to (64.0, 41.3)
- moved U4 380.5 mm to (64.0, 62.9)
- moved U5 380.5 mm to (64.0, 48.3)
- moved U6 380.5 mm to (64.0, 77.5)
- moved C901 380.5 mm to (72.3, 69.8)
- moved D901 380.5 mm to (72.9, 77.5)
- moved R901 380.5 mm to (72.3, 73.7)
- moved TP1201 352.5 mm to (23.1, 92.5)
- moved TP207 347.2 mm to (51.8, 45.7)
- moved TP206 346.0 mm to (51.6, 78.0)
- moved TP1202 346.0 mm to (23.1, 102.4)
- moved TP203 345.5 mm to (51.6, 66.8)
- moved TP209 329.6 mm to (93.7, 38.6)
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Connections:
- J3 pad 1: /MOD_OSC_RIBBON_CTL -> GND
- J3 pad 3: GND -> /MOD_OSC_RIBBON_CTL
- U4 pad 1: /ribbon_controller/gate_conditioner/GATED_CLK -> Net-(D501-Pad1)
- U4 pad 10: /ribbon_controller/gate_conditioner/GD_IN -> /ribbon_controller/gate_conditioner/GATED_CLK
- U4 pad 11: Net-(U4-Pad11) -> /ribbon_controller/gate_conditioner/S&H_TRIG
- U4 pad 12: Net-(D501-Pad1) -> /ribbon_controller/gate_conditioner/GATED_CLK
- U4 pad 13: Net-(D501-Pad1) -> Net-(U4-Pad13)
- U4 pad 2: Net-(U4-Pad2) -> Net-(D501-Pad1)
- U4 pad 3: /ribbon_controller/gate_conditioner/S&H_TRIG -> Net-(U4-Pad3)
- U4 pad 4: /ribbon_controller/gate_conditioner/GATED_CLK -> /ribbon_controller/gate_conditioner/GD_IN
- U4 pad 5: /ribbon_controller/gate_conditioner/GD_IN -> Net-(U4-Pad5)
- U4 pad 6: Net-(U4-Pad6) -> /ribbon_controller/TRIG_9
- U4 pad 8: Net-(U4-Pad8) -> /ribbon_controller/gate_conditioner/GD_IN
- U4 pad 9: /ribbon_controller/TRIG_9 -> Net-(U4-Pad9)
- U5 pad 1: Net-(U4-Pad2) -> unconnected-(U5-Pad1)
- U5 pad 11: /ribbon_controller/~{CLK_9} -> Net-(U5-Pad11)
- U5 pad 12: Net-(U4-Pad8) -> /RIBBON_GATE
- U5 pad 13: unconnected-(U5-Pad13) -> Net-(U4-Pad13)
- U5 pad 2: /RIBBON_GATE -> Net-(U4-Pad5)
- U5 pad 3: Net-(U5-Pad3) -> /ribbon_controller/~{CLK_9}
- U5 pad 6: Net-(U5-Pad6) -> Net-(U4-Pad3)
- U5 pad 8: Net-(U4-Pad11) -> Net-(U5-Pad8)
- U6 pad 10: Net-(U6-Pad10) -> Net-(U5-Pad11)
- U6 pad 11: /ribbon_controller/gate_conditioner/GATED_CLK -> /ribbon_controller/gate_conditioner/S&H_TRIG
- U6 pad 2: Net-(U4-Pad6) -> Net-(U4-Pad9)
- U6 pad 3: Net-(U4-Pad6) -> Net-(U4-Pad9)
- U6 pad 4: Net-(U5-Pad6) -> Net-(U5-Pad8)
- U6 pad 5: /ribbon_controller/gate_conditioner/S&H_TRIG -> /ribbon_controller/comparator/COMP_OUT
- U6 pad 6: Net-(U5-Pad3) -> Net-(D901-Pad2)
- U6 pad 8: Net-(D901-Pad2) -> Net-(U6-Pad8)
- U6 pad 9: /ribbon_controller/comparator/COMP_OUT -> /ribbon_controller/gate_conditioner/GATED_CLK
- U8 pad 1: Net-(D1301-Pad1) -> Net-(D1603-Pad1)
- U8 pad 10: /gate_controller/VCA_ENV_GATE -> /gate_controller/VCF_ENV_GATE
- U8 pad 11: /gate_controller/S&H_GATE -> /gate_controller/MOD_ENV_GATE
- U8 pad 12: Net-(D1601-Pad1) -> Net-(D1303-Pad1)
- U8 pad 13: Net-(D1603-Pad1) -> Net-(D1301-Pad1)
- U8 pad 2: Net-(D1303-Pad1) -> Net-(D1601-Pad1)
- U8 pad 3: /gate_controller/MOD_ENV_GATE -> /gate_controller/S&H_GATE
- U8 pad 4: /gate_controller/VCF_ENV_GATE -> /gate_controller/VCA_ENV_GATE
- U8 pad 5: Net-(D1401-Pad1) -> Net-(D1503-Pad1)
- U8 pad 6: Net-(D1403-Pad1) -> Net-(D1501-Pad1)
- U8 pad 8: Net-(D1501-Pad1) -> Net-(D1403-Pad1)
- U8 pad 9: Net-(D1503-Pad1) -> Net-(D1401-Pad1)
- U802 pad 2: Net-(U6-Pad10) -> Net-(U6-Pad8)
Routing:
- net +15V: track 0.00 -> 672.5 mm, vias 0 -> 12
- net -15V: track 0.00 -> 274.5 mm, vias 0 -> 3
- net /VCA_CV: track 0.00 -> 237.8 mm
- net /RIBBON_CV: track 0.00 -> 193.9 mm
- net /gate_controller/VCA_ADSR_gate_logic/AUTO_GATE: track 0.00 -> 181.1 mm
- net /VCF_B_RIBBON_CTL: track 0.00 -> 178.2 mm
- net Net-(D501-Pad1): track 0.00 -> 140.0 mm, vias 0 -> 3
- net /MOD_OSC_RIBBON_CTL: track 0.00 -> 139.5 mm, vias 0 -> 2
- net /RIBBON_GATE: track 0.00 -> 138.5 mm, vias 0 -> 2
- net /ribbon_controller/comparator/COMP_OUT: track 0.00 -> 136.6 mm, vias 0 -> 2
- net /VCA_ADSR: track 0.00 -> 134.0 mm, vias 0 -> 4
- net /GATE_IN: track 0.00 -> 130.9 mm, vias 0 -> 3
- net Net-(J301-Pad2): track 0.00 -> 126.7 mm, vias 0 -> 1
- net /ribbon_controller/gate_conditioner/GATED_CLK: track 0.00 -> 126.7 mm, vias 0 -> 4
- net /gate_controller/VCF_ENV_GATE: track 0.00 -> 123.3 mm, vias 0 -> 3
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- added copper zone on B.Cu, net GND
- added copper zone on F.Cu, net GND
Other:
- board outline added: 193 x 82.5 mm
