File: summer_2022_refurb/ADSR_board/kicad_6/ADSR_board.kicad_pcb (KiCad board)
At the start: 2 copper layers, 172.7 x 107.9 mm, 157 parts, among them J1 ribbon_port, J2 modosc_port, J3 VCO_port, J4 VCF_port, J5 power_entry, Q201 2N7002, Q202 MMBT3904, Q203 MMBT3904, Q204 MMBT3904, Q301 2N7002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

Commit message: Change some ADSR board values
Parts:
- R203, R210, R303, R310, R403, R410: value R -> 100
- R207, R307, R407: value R -> 680
- R211, R311, R411: value 22 -> 100
Changed lines of the file:
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@@
       (effects (font (size 1 1) (thickness 0.15)) (justify mirror))
     )
-    (fp_text value "R" (at 0 -1.65) (layer "B.Fab")
+    (fp_text value "680" (at 0 -1.65) (layer "B.Fab")
       (effects (font (size 1 1) (thickness 0.15)) (justify mirror))
     )
@@
       (effects (font (size 1 1) (thickness 0.15)) (justify mirror))
     )
-    (fp_text value "22" (at 0 -1.65) (layer "B.Fab")
+    (fp_text value "100" (at 0 -1.65) (layer "B.Fab")
       (effects (font (size 1 1) (thickness 0.15)) (justify mirror))
     )
@@
       (effects (font (size 1 1) (thickness 0.15)) (justify mirror))
     )
-    (fp_text value "R" (at 0 -1.65) (layer "B.Fab")
+    (fp_text value "100" (at 0 -1.65) (layer "B.Fab")
       (effects (font (size 1 1) (thickness 0.15)) (justify mirror))
     )
@@
       (effects (font (size 1 1) (thickness 0.15)) (justify mirror))
     )
-    (fp_text value "R" (at 0 -1.65) (layer "B.Fab")
+    (fp_text value "100" (at 0 -1.65) (layer "B.Fab")
       (effects (font (size 1 1) (thickness 0.15)) (justify mirror))
     )
@@
       (effects (font (size 1 1) (thickness 0.15)) (justify mirror))
     )
-    (fp_text value "R" (at 0 -1.65) (layer "B.Fab")
+    (fp_text value "680" (at 0 -1.65) (layer "B.Fab")
       (effects (font (size 1 1) (thickness 0.15)) (justify mirror))
     )
@@
       (effects (font (size 1 1) (thickness 0.15)) (justify mirror))
     )
-    (fp_text value "R" (at 0 -1.65) (layer "B.Fab")
+    (fp_text value "100" (at 0 -1.65) (layer "B.Fab")
       (effects (font (size 1 1) (thickness 0.15)) (justify mirror))
     )
@@
       (effects (font (size 1 1) (thickness 0.15)) (justify mirror))
     )
-    (fp_text value "R" (at 0 -1.65) (layer "B.Fab")
+    (fp_text value "100" (at 0 -1.65) (layer "B.Fab")
       (effects (font (size 1 1) (thickness 0.15)) (justify mirror))
     )
@@
       (effects (font (size 1 1) (thickness 0.15)) (justify mirror))
     )
-    (fp_text value "22" (at 0 -1.65) (layer "B.Fab")
+    (fp_text value "100" (at 0 -1.65) (layer "B.Fab")
       (effects (font (size 1 1) (thickness 0.15)) (justify mirror))
     )
@@
       (effects (font (size 1 1) (thickness 0.15)) (justify mirror))
     )
-    (fp_text value "22" (at 0 -1.65) (layer "B.Fab")
+    (fp_text value "100" (at 0 -1.65) (layer "B.Fab")
       (effects (font (size 1 1) (thickness 0.15)) (justify mirror))
     )
@@
       (effects (font (size 1 1) (thickness 0.15)) (justify mirror))
     )
-    (fp_text value "R" (at 0 -1.65) (layer "B.Fab")
+    (fp_text value "680" (at 0 -1.65) (layer "B.Fab")
       (effects (font (size 1 1) (thickness 0.15)) (justify mirror))
     )
@@
       (effects (font (size 1 1) (thickness 0.15)) (justify mirror))
     )
-    (fp_text value "R" (at 0 -1.65) (layer "B.Fab")
+    (fp_text value "100" (at 0 -1.65) (layer "B.Fab")
       (effects (font (size 1 1) (thickness 0.15)) (justify mirror))
     )
@@
       (effects (font (size 1 1) (thickness 0.15)) (justify mirror))
     )
-    (fp_text value "R" (at 0 -1.65) (layer "B.Fab")
+    (fp_text value "100" (at 0 -1.65) (layer "B.Fab")
       (effects (font (size 1 1) (thickness 0.15)) (justify mirror))
     )

Commit message: Change ADSR pot values
Parts:
- RV201, RV202, RV204, RV301, RV302, RV304, RV401, RV402, RV404: value 500kA -> 1MA
Changed lines of the file:
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@@
       (effects (font (size 1 1) (thickness 0.15)))
     )
-    (fp_text value "500kA" (at 0 9.86 90) (layer "F.Fab")
+    (fp_text value "1MA" (at 0 9.86 90) (layer "F.Fab")
       (effects (font (size 1 1) (thickness 0.15)))
     )
@@
       (effects (font (size 1 1) (thickness 0.15)))
     )
-    (fp_text value "500kA" (at 0 9.86 90) (layer "F.Fab")
+    (fp_text value "1MA" (at 0 9.86 90) (layer "F.Fab")
       (effects (font (size 1 1) (thickness 0.15)))
     )
@@
       (effects (font (size 1 1) (thickness 0.15)))
     )
-    (fp_text value "500kA" (at 0 9.86 90) (layer "F.Fab")
+    (fp_text value "1MA" (at 0 9.86 90) (layer "F.Fab")
       (effects (font (size 1 1) (thickness 0.15)))
     )
@@
       (effects (font (size 1 1) (thickness 0.15)))
     )
-    (fp_text value "500kA" (at 0 9.86 90) (layer "F.Fab")
+    (fp_text value "1MA" (at 0 9.86 90) (layer "F.Fab")
       (effects (font (size 1 1) (thickness 0.15)))
     )
@@
       (effects (font (size 1 1) (thickness 0.15)))
     )
-    (fp_text value "500kA" (at 0 9.86 90) (layer "F.Fab")
+    (fp_text value "1MA" (at 0 9.86 90) (layer "F.Fab")
       (effects (font (size 1 1) (thickness 0.15)))
     )
@@
       (effects (font (size 1 1) (thickness 0.15)))
     )
-    (fp_text value "500kA" (at 0 9.86 90) (layer "F.Fab")
+    (fp_text value "1MA" (at 0 9.86 90) (layer "F.Fab")
       (effects (font (size 1 1) (thickness 0.15)))
     )
@@
       (effects (font (size 1 1) (thickness 0.15)))
     )
-    (fp_text value "500kA" (at 0 9.86 90) (layer "F.Fab")
+    (fp_text value "1MA" (at 0 9.86 90) (layer "F.Fab")
       (effects (font (size 1 1) (thickness 0.15)))
     )
@@
       (effects (font (size 1 1) (thickness 0.15)))
     )
-    (fp_text value "500kA" (at 0 9.86 90) (layer "F.Fab")
+    (fp_text value "1MA" (at 0 9.86 90) (layer "F.Fab")
       (effects (font (size 1 1) (thickness 0.15)))
     )
@@
       (effects (font (size 1 1) (thickness 0.15)))
     )
-    (fp_text value "500kA" (at 0 9.86 90) (layer "F.Fab")
-      (effects (font (size 1 1) (thickness 0.15)))
-    )
+    (fp_text value "1MA" (at 0 9.86 90) (layer "F.Fab")
+      (effects (font (size 1 1) (thickness 0.15)))
+    )
