File: summer_2022_refurb/main_VCO_board/kicad_6/octave_divider.kicad_sch (KiCad schematic)
At the start: 10 parts, among them U2 TL074, U5 4013

Commit message: Fix VCO issues, suboct switching, component values
Connections:
- net -5V REF renamed -5V_REF
Changed lines of the file:
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@@
   (title_block
     (title "Josh Ox Ribon Synth Main VCO board")
-    (date "2022-06-18")
-    (rev "0")
+    (date "2022-07-07")
+    (rev "0.1")
     (comment 2 "creativecommons.org/licences/by/4.0")
     (comment 3 "license: CC by 4.0")
@@
     (effects (font (size 1.27 1.27)) (justify left bottom))
   )
-  (global_label "-5V REF" (shape input) (at 158.75 93.98 180) (fields_autoplaced)
+  (global_label "-5V_REF" (shape input) (at 158.75 93.98 180) (fields_autoplaced)
     (effects (font (size 1.27 1.27)) (justify right))
     (property "Intersheet References" "${INTERSHEET_REFS}" (id 0) (at 147.9912 93.9006 0)
