File: summer_2022_refurb/ribbon_board/kicad_6/ribbon_controller.kicad_sch (KiCad schematic)
At the start: 16 parts, among them SW201 SW_SPDT, U3 TL072

Commit message: Update ribbon board values
Parts:
- R201: value R -> 10k
- R202, R203, RV201: value R -> 100k
Changed lines of the file:
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@@
       (effects (font (size 1.27 1.27)) (justify left))
     )
-    (property "Value" "R" (id 1) (at 219.71 118.1099 0)
+    (property "Value" "10k" (id 1) (at 219.71 118.1099 0)
       (effects (font (size 1.27 1.27)) (justify left))
     )
@@
     (in_bom yes) (on_board yes) (fields_autoplaced)
     (property "Reference" "R203" (id 0) (at 247.65 81.28 90))
-    (property "Value" "R" (id 1) (at 247.65 83.82 90))
+    (property "Value" "100k" (id 1) (at 247.65 83.82 90))
     (property "Footprint" "Resistor_SMD:R_0805_2012Metric" (id 2) (at 247.65 89.408 90)
       (effects (font (size 1.27 1.27)) hide)
@@
     (in_bom yes) (on_board yes) (fields_autoplaced)
     (property "Reference" "R202" (id 0) (at 231.14 81.28 90))
-    (property "Value" "R" (id 1) (at 231.14 83.82 90))
+    (property "Value" "100k" (id 1) (at 231.14 83.82 90))
     (property "Footprint" "Resistor_SMD:R_0805_2012Metric" (id 2) (at 231.14 89.408 90)
       (effects (font (size 1.27 1.27)) hide)
@@
       (effects (font (size 1.27 1.27)) (justify right))
     )
-    (property "Value" "R" (id 1) (at 214.63 107.9499 0)
+    (property "Value" "100k" (id 1) (at 214.63 107.9499 0)
       (effects (font (size 1.27 1.27)) (justify right))
     )
