File: summer_2022_refurb/new_panel/kicad_6/panel_dims.kicad_pcb (KiCad board)
At the start: 2 copper layers, 602 x 322.6 mm, 79 parts, among them SW1 SR1712F-0204, SW1 SW_SPDT, SW101 SW_SPDT_MSM, SW1201 SW_SPDT, SW1301 SW_SPDT_MSM, SW1401 SW_SPDT_CO, SW1401 SW_SPDT_MSM, SW1402 SR1712F-0204, SW1501 SW_SPDT_MSM, SW1601 SW_SPDT_MSM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

Commit message: Add ribbon assembly screw holes
Other:
- board outline removed
