File: circuit_boards/sample_and_hold_board/kicad_6/sample_and_hold_board.kicad_pcb (KiCad board)
At the start: 2 copper layers, 40.6 x 203.2 mm, 107 parts, among them J1 VCO_port, J2 VCF_port, J3 ribbon_port, J4 power_entry, Q1 MMBT3904, Q2 2N3904, Q3 MMBT3904, SW1 SW_SPDT, U1 TL072, U2 TL072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

Commit message: Update some S&H board values
Parts:
- R21: value 100k -> 1M
- R3: value 100k -> 47k
- R9: value 220k -> 470k
Changed lines of the file:
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@@
   (title_block
     (title "Josh Ox Ribbon Synth Sample and Hold Board")
-    (date "2022-06-17")
+    (date "2022-07-21")
     (rev "0")
     (comment 2 "creativecommons.org/licences/by/4.0")
@@
       (effects (font (size 1 1) (thickness 0.15)) (justify mirror))
     )
-    (fp_text value "100k" (at 0 -1.65) (layer "B.Fab")
+    (fp_text value "1M" (at 0 -1.65) (layer "B.Fab")
       (effects (font (size 1 1) (thickness 0.15)) (justify mirror))
     )
@@
       (effects (font (size 1 1) (thickness 0.15)) (justify mirror))
     )
-    (fp_text value "100k" (at 0 -1.65) (layer "B.Fab")
+    (fp_text value "47k" (at 0 -1.65) (layer "B.Fab")
       (effects (font (size 1 1) (thickness 0.15)) (justify mirror))
     )
@@
       (effects (font (size 1 1) (thickness 0.15)) (justify mirror))
     )
-    (fp_text value "220k" (at 0 -1.65) (layer "B.Fab")
+    (fp_text value "470k" (at 0 -1.65) (layer "B.Fab")
       (effects (font (size 1 1) (thickness 0.15)) (justify mirror))
     )
