File: circuit_boards/mod_osc_board/kicad_6/level_shifter.kicad_sch (KiCad schematic)
At the start: 4 parts, among them U202 TL072

Commit message: Update some mod-osc board values
Parts:
- R301: value 100k -> 47k
Changed lines of the file:
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@@
   (title_block
     (title "Josh Ox Ribbon Synth Mod Osc board")
-    (date "2022-06-17")
+    (date "2022-07-21")
     (rev "0")
     (comment 2 "creativecommons.org/licences/by/4.0")
@@
     (in_bom yes) (on_board yes) (fields_autoplaced)
     (property "Reference" "R301" (id 0) (at 132.08 95.25 90))
-    (property "Value" "100k" (id 1) (at 132.08 97.79 90))
+    (property "Value" "47k" (id 1) (at 132.08 97.79 90))
     (property "Footprint" "Resistor_SMD:R_0805_2012Metric" (id 2) (at 132.08 103.378 90)
       (effects (font (size 1.27 1.27)) hide)
