File: circuit_boards/VCF_VCA_board/kicad_6/VCA.kicad_sch (KiCad schematic)
At the start: 22 parts, among them U10 SSI2164, U11 SSI2164, U6 TL072, U7 TL072

Commit message: Update some VCF board values
Parts:
- D401, D402: value D_Zener -> 2v4
Changed lines of the file:
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@@
   (title_block
     (title "Josh Ox Ribbon Synth VCF/VCA board")
-    (date "2022-06-16")
+    (date "2022-07-21")
     (rev "0")
     (comment 1 "creativecommons.org/licenses/by/4.0/")
@@
       (effects (font (size 1.27 1.27)) (justify right))
     )
-    (property "Value" "D_Zener" (id 1) (at 209.55 91.4399 90)
+    (property "Value" "2v4" (id 1) (at 209.55 91.4399 90)
       (effects (font (size 1.27 1.27)) (justify right))
     )
@@
       (effects (font (size 1.27 1.27)) (justify left))
     )
-    (property "Value" "D_Zener" (id 1) (at 209.55 81.2799 90)
+    (property "Value" "2v4" (id 1) (at 209.55 81.2799 90)
       (effects (font (size 1.27 1.27)) (justify left))
     )

Commit message: Change VCA R for smoother volume knob action
Parts:
- R407: value 2M2 -> 10M
Changed lines of the file:
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@@
     (in_bom yes) (on_board yes)
     (property "Reference" "R407" (id 0) (at 85.09 110.49 90))
-    (property "Value" "2M2" (id 1) (at 85.09 113.03 90))
+    (property "Value" "10M" (id 1) (at 85.09 113.03 90))
     (property "Footprint" "Resistor_SMD:R_0805_2012Metric" (id 2) (at 85.09 117.348 90)
       (effects (font (size 1.27 1.27)) hide)
