File: circuit_boards/ribbon_uC/kicad_7/ribbon_board.kicad_pcb (KiCad board)
At the start: 4 copper layers, 193 x 69.8 mm, 166 parts, among them J1 VCO_port, J2 VCF_port, J201 SWD_header, J3 mod_osc_port, J4 ADSR_port, J5 S&H_port, J6 ext_port, J7 power_entry, J8 MIDI_IO_port, SW201 SW_SPDT_MSM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

Commit message: Change value of ribbon scaler R for 1v/oct trimming
Parts:
- R301, R302, R303, R304: value 4k7 -> 15k
Changed lines of the file:
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@@
         (effects (font (size 1 1) (thickness 0.15)) (justify mirror))
     )
-    (fp_text value "4k7" (at 0 -1.65) (layer "B.Fab")
+    (fp_text value "15k" (at 0 -1.65) (layer "B.Fab")
         (effects (font (size 1 1) (thickness 0.15)) (justify mirror))
     )
@@
         (effects (font (size 1 1) (thickness 0.15)) (justify mirror))
     )
-    (fp_text value "4k7" (at 0 -1.65) (layer "B.Fab")
+    (fp_text value "15k" (at 0 -1.65) (layer "B.Fab")
         (effects (font (size 1 1) (thickness 0.15)) (justify mirror))
     )
@@
         (effects (font (size 1 1) (thickness 0.15)) (justify mirror))
     )
-    (fp_text value "4k7" (at 0 -1.65 180) (layer "B.Fab")
+    (fp_text value "15k" (at 0 -1.65 180) (layer "B.Fab")
         (effects (font (size 1 1) (thickness 0.15)) (justify mirror))
     )
@@
         (effects (font (size 1 1) (thickness 0.15)) (justify mirror))
     )
-    (fp_text value "4k7" (at 0 -1.65 180) (layer "B.Fab")
+    (fp_text value "15k" (at 0 -1.65 180) (layer "B.Fab")
         (effects (font (size 1 1) (thickness 0.15)) (justify mirror))
     )
